Commit message: Changed for Humbe (branch)

File: src/daadbot_desc/urdf/daadbot.urdf.xacro (robot description, xacro)
@@ -5,6 +5,6 @@
   <xacro:include filename = "$(find daadbot_desc)/urdf/daadbot_ros2_control.xacro"/>
   <xacro:property name='PI' value='3.141592653589793'/>
-  <xacro:property name='velocity' value='10.0'/>
-  <xacro:property name='effort' value='30.0'/>
+  <xacro:property name='velocity' value='20.0'/>
+  <xacro:property name='effort' value='300.0'/>
   <link name="world"/>
   <joint
@@ -345,5 +345,5 @@
   </joint>
   <link
-    name="link_6">
+    name="Link_6">
     <inertial>
       <origin
@@ -393,5 +393,5 @@
       link="Link_5" />
     <child
-      link="link_6" />
+      link="Link_6" />
     <axis
       xyz="0 0 1" />
@@ -449,5 +449,5 @@
       rpy="-1.5707963267949 0 3.14159265358979" />
     <parent
-      link="link_6" />
+      link="Link_6" />
     <child
       link="Link_7" />
@@ -572,4 +572,75 @@
   </joint>
   <link
+    name="base_claw_link1">
+    <inertial>
+      <origin
+        xyz="-1.058E-05 -0.015556 -0.00071484"
+        rpy="0 0 0" />
+      <mass
+        value="0.0011042" />
+      <inertia
+        ixx="1.5467E-07"
+        ixy="-7.9881E-10"
+        ixz="-2.9739E-11"
+        iyy="3.5247E-09"
+        iyz="7.7059E-09"
+        izz="1.5576E-07" />
+    </inertial>
+    <visual>
+      <origin
+        xyz="0 0 0"
+        rpy="0 0 0" />
+      <geometry>
+        <mesh
+          filename="package://daadbot_desc/meshes/base_claw_link1.STL" />
+      </geometry>
+      <material
+        name="">
+        <color
+          rgba="1 1 1 1" />
+      </material>
+    </visual>
+    <collision>
+      <origin
+        xyz="0 0 0"
+        rpy="0 0 0" />
+      <geometry>
+        <mesh
+          filename="package://daadbot_desc/meshes/base_claw_link1.STL" />
+      </geometry>
+    </collision>
+  </link>
+  <joint
+    name="base_claw_joint1_mimic"
+    type="fixed">
+    <parent
+      link="Link_7" />
+    <child
+      link="dummy_base_claw_joint1_mimic" />
+  </joint>
+  <link name="dummy_base_claw_joint1_mimic"/>
+  <joint
+    name="base_claw_joint1"
+    type="revolute">
+    <origin
+      xyz="-0.00548036760308535 0.0047463745042049 0.0685789689085226"
+      rpy="-1.52010273242897 0 0" />
+    <parent
+      link="Link_7" />
+    <child
+      link="base_claw_link1" />
+    <axis
+      xyz="0.0472460759822863 -0.0506152984712078 -0.997600070100712" />
+    <limit
+      lower="0"
+      upper="0.9"
+      effort="${effort}"
+      velocity="${velocity}" />
+    <mimic
+      joint="gear1_joint"
+      multiplier="-1"
+      offset="0" />
+  </joint>
+  <link
     name="gear1_claw">
     <inertial>
@@ -612,4 +683,13 @@
   </link>
   <joint
+    name="claw_joint1_mimic"
+    type="fixed">
+    <parent
+      link="gear1" />
+    <child
+      link="dummy_claw_joint1_mimic" />
+  </joint>
+  <link name="dummy_claw_joint1_mimic"/>
+  <joint
     name="claw_joint1"
     type="revolute">
@@ -674,4 +754,13 @@
   </link>
   <joint
+    name="gear2_joint_mimic"
+    type="fixed">
+    <parent
+      link="endeffector" />
+    <child
+      link="dummy_gear2_joint_mimic" />
+  </joint>
+  <link name="dummy_gear2_joint_mimic"/>
+  <joint
     name="gear2_joint"
     type="revolute">
@@ -685,4 +774,75 @@
     <axis
       xyz="-0.0472460759822667 0.0506152984712492 0.997600070100711" />
+    <limit
+      lower="0"
+      upper="0.9"
+      effort="${effort}"
+      velocity="${velocity}" />
+    <mimic
+      joint="gear1_joint"
+      multiplier="-1"
+      offset="0" />
+  </joint>
+  <link
+    name="base_claw_link2">
+    <inertial>
+      <origin
+        xyz="0.00030048 -0.015554 -0.00070023"
+        rpy="0 0 0" />
+      <mass
+        value="0.0011042" />
+      <inertia
+        ixx="1.5464E-07"
+        ixy="2.238E-09"
+        ixz="-1.8519E-10"
+        iyy="3.5683E-09"
+        iyz="7.8475E-09"
+        izz="1.5574E-07" />
+    </inertial>
+    <visual>
+      <origin
+        xyz="0 0 0"
+        rpy="0 0 0" />
+      <geometry>
+        <mesh
+          filename="package://daadbot_desc/meshes/base_claw_link2.STL" />
+      </geometry>
+      <material
+        name="">
+        <color
+          rgba="1 1 1 1" />
+      </material>
+    </visual>
+    <collision>
+      <origin
+        xyz="0 0 0"
+        rpy="0 0 0" />
+      <geometry>
+        <mesh
+          filename="package://daadbot_desc/meshes/base_claw_link2.STL" />
+      </geometry>
+    </collision>
+  </link>
+  <joint
+    name="base_claw_joint2_mimic"
+    type="fixed">
+    <parent
+      link="Link_7" />
+    <child
+      link="dummy_base_claw_joint2_mimic" />
+  </joint>
+  <link name="dummy_base_claw_joint2_mimic"/>
+  <joint
+    name="base_claw_joint2"
+    type="revolute">
+    <origin
+      xyz="0.00500790684313079 0.00524245830200445 0.0685789689082188"
+      rpy="-1.52010273242897 0 0" />
+    <parent
+      link="Link_7" />
+    <child
+      link="base_claw_link2" />
+    <axis
+      xyz="-0.0472460759822792 0.0506152984712578 0.99760007010071" />
     <limit
       lower="0"
@@ -736,4 +896,13 @@
   </link>
   <joint
+    name="claw_joint2_mimic"
+    type="fixed">
+    <parent
+      link="gear2_link" />
+    <child
+      link="dummy_claw_joint2_mimic" />
+  </joint>
+  <link name="dummy_claw_joint2_mimic"/>
+  <joint
     name="claw_joint2"
     type="revolute">
@@ -757,127 +926,3 @@
       offset="0" />
   </joint>
-  <link
-    name="base_claw_link2">
-    <inertial>
-      <origin
-        xyz="0.00030048 -0.015554 -0.00070023"
-        rpy="0 0 0" />
-      <mass
-        value="0.0011042" />
-      <inertia
-        ixx="1.5464E-07"
-        ixy="2.238E-09"
-        ixz="-1.8519E-10"
-        iyy="3.5683E-09"
-        iyz="7.8475E-09"
-        izz="1.5574E-07" />
-    </inertial>
-    <visual>
-      <origin
-        xyz="0 0 0"
-        rpy="0 0 0" />
-      <geometry>
-        <mesh
-          filename="package://daadbot_desc/meshes/base_claw_link2.STL" />
-      </geometry>
-      <material
-        name="">
-        <color
-          rgba="1 1 1 1" />
-      </material>
-    </visual>
-    <collision>
-      <origin
-        xyz="0 0 0"
-        rpy="0 0 0" />
-      <geometry>
-        <mesh
-          filename="package://daadbot_desc/meshes/base_claw_link2.STL" />
-      </geometry>
-    </collision>
-  </link>
-  <joint
-    name="base_claw_joint2"
-    type="revolute">
-    <origin
-      xyz="0.00500790684313079 0.00524245830200445 0.0685789689082188"
-      rpy="-1.52010273242897 0 0" />
-    <parent
-      link="Link_7" />
-    <child
-      link="base_claw_link2" />
-    <axis
-      xyz="-0.0472460759822792 0.0506152984712578 0.99760007010071" />
-    <limit
-      lower="0"
-      upper="0.9"
-      effort="${effort}"
-      velocity="${velocity}" />
-    <mimic
-      joint="gear1_joint"
-      multiplier="-1"
-      offset="0" />
-  </joint>
-  <link
-    name="base_claw_link1">
-    <inertial>
-      <origin
-        xyz="-1.058E-05 -0.015556 -0.00071484"
-        rpy="0 0 0" />
-      <mass
-        value="0.0011042" />
-      <inertia
-        ixx="1.5467E-07"
-        ixy="-7.9881E-10"
-        ixz="-2.9739E-11"
-        iyy="3.5247E-09"
-        iyz="7.7059E-09"
-        izz="1.5576E-07" />
-    </inertial>
-    <visual>
-      <origin
-        xyz="0 0 0"
-        rpy="0 0 0" />
-      <geometry>
-        <mesh
-          filename="package://daadbot_desc/meshes/base_claw_link1.STL" />
-      </geometry>
-      <material
-        name="">
-        <color
-          rgba="1 1 1 1" />
-      </material>
-    </visual>
-    <collision>
-      <origin
-        xyz="0 0 0"
-        rpy="0 0 0" />
-      <geometry>
-        <mesh
-          filename="package://daadbot_desc/meshes/base_claw_link1.STL" />
-      </geometry>
-    </collision>
-  </link>
-  <joint
-    name="base_claw_joint1"
-    type="revolute">
-    <origin
-      xyz="-0.00548036760308535 0.0047463745042049 0.0685789689085226"
-      rpy="-1.52010273242897 0 0" />
-    <parent
-      link="Link_7" />
-    <child
-      link="base_claw_link1" />
-    <axis
-      xyz="0.0472460759822863 -0.0506152984712078 -0.997600070100712" />
-    <limit
-      lower="0"
-      upper="0.9"
-      effort="${effort}"
-      velocity="${velocity}" />
-    <mimic
-      joint="gear1_joint"
-      multiplier="-1"
-      offset="0" />
-  </joint>
 </robot>

File: src/daadbot_desc/urdf/daadbot_ros2_control.xacro (robot description, xacro)
@@ -19,4 +19,6 @@
             </command_interface>
             <state_interface name="position"/>
+            <state_interface name="velocity"/>
+            <state_interface name="effort"/>
         </joint>
         <joint name="joint_2">
@@ -26,4 +28,6 @@
             </command_interface>
             <state_interface name="position"/>
+            <state_interface name="velocity"/>
+            <state_interface name="effort"/>
         </joint>
         <joint name="joint_3">
@@ -33,4 +37,6 @@
             </command_interface>
             <state_interface name="position"/>
+            <state_interface name="velocity"/>
+            <state_interface name="effort"/>
         </joint>
         <joint name="joint_4">
@@ -40,4 +46,6 @@
             </command_interface>
             <state_interface name="position"/>
+            <state_interface name="velocity"/>
+            <state_interface name="effort"/>
         </joint>
         <joint name="joint_5">
@@ -47,4 +55,6 @@
             </command_interface>
             <state_interface name="position"/>
+            <state_interface name="velocity"/>
+            <state_interface name="effort"/>
         </joint>
         <joint name="joint_6">
@@ -54,4 +64,6 @@
             </command_interface>
             <state_interface name="position"/>
+            <state_interface name="velocity"/>
+            <state_interface name="effort"/>
         </joint>
         <joint name="joint_7">
@@ -61,4 +73,6 @@
             </command_interface>
             <state_interface name="position"/>
+            <state_interface name="velocity"/>
+            <state_interface name="effort"/>
         </joint>
         <joint name="gear1_joint">
@@ -68,8 +82,13 @@
             </command_interface>
             <state_interface name="position"/>
+            <state_interface name="velocity"/>
+            <state_interface name="effort"/>
         </joint>
         <joint name="base_claw_joint1">
             <param name="mimic">gear1_joint</param>
             <param name="multiplier">-1</param>
+            <state_interface name="position"/>
+            <state_interface name="velocity"/>
+            <state_interface name="effort"/>
         </joint>
         <joint name="claw_joint1">
@@ -77,16 +96,27 @@
             <param name="multiplier">1</param>
             <state_interface name="position"/>
+            <state_interface name="velocity"/>
+            <state_interface name="effort"/>
         </joint>
         <joint name="gear2_joint">
             <param name="mimic">gear1_joint</param>
             <param name="multiplier">-1</param>
+            <state_interface name="position"/>
+            <state_interface name="velocity"/>
+            <state_interface name="effort"/>
         </joint>
         <joint name="base_claw_joint2">
             <param name="mimic">gear1_joint</param>
             <param name="multiplier">-1</param>
+            <state_interface name="position"/>
+            <state_interface name="velocity"/>
+            <state_interface name="effort"/>
         </joint>
         <joint name="claw_joint2">
             <param name="mimic">base_claw_joint2</param>
             <param name="multiplier">-1</param>
+            <state_interface name="position"/>
+            <state_interface name="velocity"/>
+            <state_interface name="effort"/>
         </joint>
     </ros2_control>

Commit message: Changed effort limits to 300 from 30.

File: src/daadbot_desc/urdf/daadbot.urdf.xacro (robot description, xacro)
@@ -6,5 +6,5 @@
   <xacro:property name='PI' value='3.141592653589793'/>
   <xacro:property name='velocity' value='10.0'/>
-  <xacro:property name='effort' value='30.0'/>
+  <xacro:property name='effort' value='300.0'/>
   <link name="world"/>
   <joint
