Commit message: Made some changes for humble. (.h instead of .hpp)

File: src/daadbot_desc/urdf/daadbotrviz.urdf.xacro (robot description, xacro)
@@ -3,5 +3,5 @@
   <xacro:property name='PI' value='3.141592653589793'/>
   <xacro:property name='velocity' value='10.0'/>
-  <xacro:property name='effort' value='30.0'/>
+  <xacro:property name='effort' value='300.0'/>
   <link name="world"/>
   <joint

File: src/daadbot_desc/urdf/urdf_oct/daadbot.urdf.xacro (robot description, xacro)
@@ -1,9 +1,9 @@
 <?xml version="1.0" encoding="utf-8"?>
 <robot xmlns:xacro="http://www.ros.org/wiki/xacro" name="daadbot">
-  <xacro:arg name = "is_ignition" default="false"/>
+  <xacro:arg name = "is_ignition" default="true"/>
   <xacro:include filename = "$(find daadbot_desc)/urdf/urdf_oct/daadbot_gazebo.xacro"/>
   <xacro:include filename = "$(find daadbot_desc)/urdf/urdf_oct/daadbot_ros2_control.xacro"/>
   <xacro:property name='PI' value='3.141592653589793'/>
-  <xacro:property name='velocity' value='10.0'/>
+  <xacro:property name='velocity' value='20.0'/>
   <xacro:property name='effort' value='300.0'/>
   <link name="world"/>
@@ -96,5 +96,5 @@
   <joint
     name="joint_1"
-    type="revolute">
+    type="continuous">
     <origin
       xyz="0 0 0.05"
@@ -107,6 +107,6 @@
       xyz="0 0 -1" />
     <limit
-      lower="-${pi}"
-      upper="${pi}"
+      lower="0"
+      upper="3.14"
       effort="${effort}"
       velocity="${velocity}" />
@@ -212,5 +212,5 @@
   <joint
     name="joint_3"
-    type="revolute">
+    type="continuous">
     <origin
       xyz="0.000359289684152012 0.435033961918617 0.0294474762975983"
@@ -223,6 +223,6 @@
       xyz="0 0 -1" />
     <limit
-      lower="-${pi}"
-      upper="${pi}"
+      lower="0"
+      upper="3.14"
       effort="${effort}"
       velocity="${velocity}" />
@@ -328,5 +328,5 @@
   <joint
     name="joint_5"
-    type="revolute">
+    type="continuous">
     <origin
       xyz="0.419299903678905 0 -0.0294999999999992"
@@ -339,6 +339,6 @@
       xyz="0 0 -1" />
     <limit
-      lower="-${pi}"
-      upper="${pi}"
+      lower="0"
+      upper="3.14"
       effort="${effort}"
       velocity="${velocity}" />
@@ -397,6 +397,6 @@
       xyz="0 0 1" />
     <limit
-      lower="-${pi}"
-      upper="0.0001"
+      lower="-3.14"
+      upper="0"
       effort="${effort}"
       velocity="${velocity}" />
@@ -444,5 +444,5 @@
   <joint
     name="joint_7"
-    type="revolute">
+    type="continuous">
     <origin
       xyz="0 -0.0909999036788988 -0.0244999999999991"
@@ -455,6 +455,6 @@
       xyz="0 0 -1" />
     <limit
-      lower="-${pi}"
-      upper="${pi}"
+      lower="0"
+      upper="3.14"
       effort="${effort}"
       velocity="${velocity}" />
@@ -572,4 +572,75 @@
   </joint>
   <link
+    name="base_claw_link1">
+    <inertial>
+      <origin
+        xyz="-1.058E-05 -0.015556 -0.00071484"
+        rpy="0 0 0" />
+      <mass
+        value="0.0011042" />
+      <inertia
+        ixx="1.5467E-07"
+        ixy="-7.9881E-10"
+        ixz="-2.9739E-11"
+        iyy="3.5247E-09"
+        iyz="7.7059E-09"
+        izz="1.5576E-07" />
+    </inertial>
+    <visual>
+      <origin
+        xyz="0 0 0"
+        rpy="0 0 0" />
+      <geometry>
+        <mesh
+          filename="package://daadbot_desc/meshes/base_claw_link1.STL" />
+      </geometry>
+      <material
+        name="">
+        <color
+          rgba="1 1 1 1" />
+      </material>
+    </visual>
+    <collision>
+      <origin
+        xyz="0 0 0"
+        rpy="0 0 0" />
+      <geometry>
+        <mesh
+          filename="package://daadbot_desc/meshes/base_claw_link1.STL" />
+      </geometry>
+    </collision>
+  </link>
+  <joint
+    name="base_claw_joint1_mimic"
+    type="fixed">
+    <parent
+      link="Link_7" />
+    <child
+      link="dummy_base_claw_joint1_mimic" />
+  </joint>
+  <link name="dummy_base_claw_joint1_mimic"/>
+  <joint
+    name="base_claw_joint1"
+    type="revolute">
+    <origin
+      xyz="-0.00548036760308535 0.0047463745042049 0.0685789689085226"
+      rpy="-1.52010273242897 0 0" />
+    <parent
+      link="Link_7" />
+    <child
+      link="base_claw_link1" />
+    <axis
+      xyz="0.0472460759822863 -0.0506152984712078 -0.997600070100712" />
+    <limit
+      lower="0"
+      upper="0.9"
+      effort="${effort}"
+      velocity="${velocity}" />
+    <mimic
+      joint="gear1_joint"
+      multiplier="-1"
+      offset="0" />
+  </joint>
+  <link
     name="gear1_claw">
     <inertial>
@@ -612,4 +683,13 @@
   </link>
   <joint
+    name="claw_joint1_mimic"
+    type="fixed">
+    <parent
+      link="gear1" />
+    <child
+      link="dummy_claw_joint1_mimic" />
+  </joint>
+  <link name="dummy_claw_joint1_mimic"/>
+  <joint
     name="claw_joint1"
     type="revolute">
@@ -674,4 +754,13 @@
   </link>
   <joint
+    name="gear2_joint_mimic"
+    type="fixed">
+    <parent
+      link="endeffector" />
+    <child
+      link="dummy_gear2_joint_mimic" />
+  </joint>
+  <link name="dummy_gear2_joint_mimic"/>
+  <joint
     name="gear2_joint"
     type="revolute">
@@ -685,4 +774,75 @@
     <axis
       xyz="-0.0472460759822667 0.0506152984712492 0.997600070100711" />
+    <limit
+      lower="0"
+      upper="0.9"
+      effort="${effort}"
+      velocity="${velocity}" />
+    <mimic
+      joint="gear1_joint"
+      multiplier="-1"
+      offset="0" />
+  </joint>
+  <link
+    name="base_claw_link2">
+    <inertial>
+      <origin
+        xyz="0.00030048 -0.015554 -0.00070023"
+        rpy="0 0 0" />
+      <mass
+        value="0.0011042" />
+      <inertia
+        ixx="1.5464E-07"
+        ixy="2.238E-09"
+        ixz="-1.8519E-10"
+        iyy="3.5683E-09"
+        iyz="7.8475E-09"
+        izz="1.5574E-07" />
+    </inertial>
+    <visual>
+      <origin
+        xyz="0 0 0"
+        rpy="0 0 0" />
+      <geometry>
+        <mesh
+          filename="package://daadbot_desc/meshes/base_claw_link2.STL" />
+      </geometry>
+      <material
+        name="">
+        <color
+          rgba="1 1 1 1" />
+      </material>
+    </visual>
+    <collision>
+      <origin
+        xyz="0 0 0"
+        rpy="0 0 0" />
+      <geometry>
+        <mesh
+          filename="package://daadbot_desc/meshes/base_claw_link2.STL" />
+      </geometry>
+    </collision>
+  </link>
+  <joint
+    name="base_claw_joint2_mimic"
+    type="fixed">
+    <parent
+      link="Link_7" />
+    <child
+      link="dummy_base_claw_joint2_mimic" />
+  </joint>
+  <link name="dummy_base_claw_joint2_mimic"/>
+  <joint
+    name="base_claw_joint2"
+    type="revolute">
+    <origin
+      xyz="0.00500790684313079 0.00524245830200445 0.0685789689082188"
+      rpy="-1.52010273242897 0 0" />
+    <parent
+      link="Link_7" />
+    <child
+      link="base_claw_link2" />
+    <axis
+      xyz="-0.0472460759822792 0.0506152984712578 0.99760007010071" />
     <limit
       lower="0"
@@ -736,4 +896,13 @@
   </link>
   <joint
+    name="claw_joint2_mimic"
+    type="fixed">
+    <parent
+      link="gear2_link" />
+    <child
+      link="dummy_claw_joint2_mimic" />
+  </joint>
+  <link name="dummy_claw_joint2_mimic"/>
+  <joint
     name="claw_joint2"
     type="revolute">
@@ -757,127 +926,3 @@
       offset="0" />
   </joint>
-  <link
-    name="base_claw_link2">
-    <inertial>
-      <origin
-        xyz="0.00030048 -0.015554 -0.00070023"
-        rpy="0 0 0" />
-      <mass
-        value="0.0011042" />
-      <inertia
-        ixx="1.5464E-07"
-        ixy="2.238E-09"
-        ixz="-1.8519E-10"
-        iyy="3.5683E-09"
-        iyz="7.8475E-09"
-        izz="1.5574E-07" />
-    </inertial>
-    <visual>
-      <origin
-        xyz="0 0 0"
-        rpy="0 0 0" />
-      <geometry>
-        <mesh
-          filename="package://daadbot_desc/meshes/base_claw_link2.STL" />
-      </geometry>
-      <material
-        name="">
-        <color
-          rgba="1 1 1 1" />
-      </material>
-    </visual>
-    <collision>
-      <origin
-        xyz="0 0 0"
-        rpy="0 0 0" />
-      <geometry>
-        <mesh
-          filename="package://daadbot_desc/meshes/base_claw_link2.STL" />
-      </geometry>
-    </collision>
-  </link>
-  <joint
-    name="base_claw_joint2"
-    type="revolute">
-    <origin
-      xyz="0.00500790684313079 0.00524245830200445 0.0685789689082188"
-      rpy="-1.52010273242897 0 0" />
-    <parent
-      link="Link_7" />
-    <child
-      link="base_claw_link2" />
-    <axis
-      xyz="-0.0472460759822792 0.0506152984712578 0.99760007010071" />
-    <limit
-      lower="0"
-      upper="0.9"
-      effort="${effort}"
-      velocity="${velocity}" />
-    <mimic
-      joint="gear1_joint"
-      multiplier="-1"
-      offset="0" />
-  </joint>
-  <link
-    name="base_claw_link1">
-    <inertial>
-      <origin
-        xyz="-1.058E-05 -0.015556 -0.00071484"
-        rpy="0 0 0" />
-      <mass
-        value="0.0011042" />
-      <inertia
-        ixx="1.5467E-07"
-        ixy="-7.9881E-10"
-        ixz="-2.9739E-11"
-        iyy="3.5247E-09"
-        iyz="7.7059E-09"
-        izz="1.5576E-07" />
-    </inertial>
-    <visual>
-      <origin
-        xyz="0 0 0"
-        rpy="0 0 0" />
-      <geometry>
-        <mesh
-          filename="package://daadbot_desc/meshes/base_claw_link1.STL" />
-      </geometry>
-      <material
-        name="">
-        <color
-          rgba="1 1 1 1" />
-      </material>
-    </visual>
-    <collision>
-      <origin
-        xyz="0 0 0"
-        rpy="0 0 0" />
-      <geometry>
-        <mesh
-          filename="package://daadbot_desc/meshes/base_claw_link1.STL" />
-      </geometry>
-    </collision>
-  </link>
-  <joint
-    name="base_claw_joint1"
-    type="revolute">
-    <origin
-      xyz="-0.00548036760308535 0.0047463745042049 0.0685789689085226"
-      rpy="-1.52010273242897 0 0" />
-    <parent
-      link="Link_7" />
-    <child
-      link="base_claw_link1" />
-    <axis
-      xyz="0.0472460759822863 -0.0506152984712078 -0.997600070100712" />
-    <limit
-      lower="0"
-      upper="0.9"
-      effort="${effort}"
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
File: src/daadbot_desc/urdf/urdf_oct_effort/daadbot.urdf.xacro (robot description, xacro)
@@ -5,5 +5,5 @@
   <xacro:include filename = "$(find daadbot_desc)/urdf/urdf_oct_effort/daadbot_ros2_control.xacro"/>
   <xacro:property name='PI' value='3.141592653589793'/>
-  <xacro:property name='velocity' value='30.0'/>
+  <xacro:property name='velocity' value='20.0'/>
   <xacro:property name='effort' value='300.0'/>
   <link name="world"/>
@@ -96,5 +96,5 @@
   <joint
     name="joint_1"
-    type="revolute">
+    type="continuous">
     <origin
       xyz="0 0 0.05"
@@ -107,6 +107,6 @@
       xyz="0 0 -1" />
     <limit
-      lower="-${pi}"
-      upper="${pi}"
+      lower="0"
+      upper="3.14"
       effort="${effort}"
       velocity="${velocity}" />
@@ -212,5 +212,5 @@
   <joint
     name="joint_3"
-    type="revolute">
+    type="continuous">
     <origin
       xyz="0.000359289684152012 0.435033961918617 0.0294474762975983"
@@ -223,6 +223,6 @@
       xyz="0 0 -1" />
     <limit
-      lower="-${pi}"
-      upper="${pi}"
+      lower="0"
+      upper="3.14"
       effort="${effort}"
       velocity="${velocity}" />
@@ -328,5 +328,5 @@
   <joint
     name="joint_5"
-    type="revolute">
+    type="continuous">
     <origin
       xyz="0.419299903678905 0 -0.0294999999999992"
@@ -339,6 +339,6 @@
       xyz="0 0 -1" />
     <limit
-      lower="-${pi}"
-      upper="${pi}"
+      lower="0"
+      upper="3.14"
       effort="${effort}"
       velocity="${velocity}" />
@@ -397,6 +397,6 @@
       xyz="0 0 1" />
     <limit
-      lower="-${pi}"
-      upper="0.001"
+      lower="-3.14"
+      upper="0"
       effort="${effort}"
       velocity="${velocity}" />
@@ -444,5 +444,5 @@
   <joint
     name="joint_7"
-    type="revolute">
+    type="continuous">
     <origin
       xyz="0 -0.0909999036788988 -0.0244999999999991"
@@ -455,6 +455,6 @@
       xyz="0 0 -1" />
     <limit
-      lower="-${pi}"
-      upper="${pi}"
+      lower="0"
+      upper="3.14"
       effort="${effort}"
       velocity="${velocity}" />
@@ -572,4 +572,75 @@
   </joint>
   <link
+    name="base_claw_link1">
+    <inertial>
+      <origin
+        xyz="-1.058E-05 -0.015556 -0.00071484"
+        rpy="0 0 0" />
+      <mass
+        value="0.0011042" />
+      <inertia
+        ixx="1.5467E-07"
+        ixy="-7.9881E-10"
+        ixz="-2.9739E-11"
+        iyy="3.5247E-09"
+        iyz="7.7059E-09"
+        izz="1.5576E-07" />
+    </inertial>
+    <visual>
+      <origin
+        xyz="0 0 0"
+        rpy="0 0 0" />
+      <geometry>
+        <mesh
+          filename="package://daadbot_desc/meshes/base_claw_link1.STL" />
+      </geometry>
+      <material
+        name="">
+        <color
+          rgba="1 1 1 1" />
+      </material>
+    </visual>
+    <collision>
+      <origin
+        xyz="0 0 0"
+        rpy="0 0 0" />
+      <geometry>
+        <mesh
+          filename="package://daadbot_desc/meshes/base_claw_link1.STL" />
+      </geometry>
+    </collision>
+  </link>
+  <joint
+    name="base_claw_joint1_mimic"
+    type="fixed">
+    <parent
+      link="Link_7" />
+    <child
+      link="dummy_base_claw_joint1_mimic" />
+  </joint>
+  <link name="dummy_base_claw_joint1_mimic"/>
+  <joint
+    name="base_claw_joint1"
+    type="revolute">
+    <origin
+      xyz="-0.00548036760308535 0.0047463745042049 0.0685789689085226"
+      rpy="-1.52010273242897 0 0" />
+    <parent
+      link="Link_7" />
+    <child
+      link="base_claw_link1" />
+    <axis
+      xyz="0.0472460759822863 -0.0506152984712078 -0.997600070100712" />
+    <limit
+      lower="0"
+      upper="0.9"
+      effort="${effort}"
+      velocity="${velocity}" />
+    <mimic
+      joint="gear1_joint"
+      multiplier="-1"
+      offset="0" />
+  </joint>
+  <link
     name="gear1_claw">
     <inertial>
@@ -612,4 +683,13 @@
   </link>
   <joint
+    name="claw_joint1_mimic"
+    type="fixed">
+    <parent
+      link="gear1" />
+    <child
+      link="dummy_claw_joint1_mimic" />
+  </joint>
+  <link name="dummy_claw_joint1_mimic"/>
+  <joint
     name="claw_joint1"
     type="revolute">
@@ -674,4 +754,13 @@
   </link>
   <joint
+    name="gear2_joint_mimic"
+    type="fixed">
+    <parent
+      link="endeffector" />
+    <child
+      link="dummy_gear2_joint_mimic" />
+  </joint>
+  <link name="dummy_gear2_joint_mimic"/>
+  <joint
     name="gear2_joint"
     type="revolute">
@@ -685,4 +774,75 @@
     <axis
       xyz="-0.0472460759822667 0.0506152984712492 0.997600070100711" />
+    <limit
+      lower="0"
+      upper="0.9"
+      effort="${effort}"
+      velocity="${velocity}" />
+    <mimic
+      joint="gear1_joint"
+      multiplier="-1"
+      offset="0" />
+  </joint>
+  <link
+    name="base_claw_link2">
+    <inertial>
+      <origin
+        xyz="0.00030048 -0.015554 -0.00070023"
+        rpy="0 0 0" />
+      <mass
+        value="0.0011042" />
+      <inertia
+        ixx="1.5464E-07"
+        ixy="2.238E-09"
+        ixz="-1.8519E-10"
+        iyy="3.5683E-09"
+        iyz="7.8475E-09"
+        izz="1.5574E-07" />
+    </inertial>
+    <visual>
+      <origin
+        xyz="0 0 0"
+        rpy="0 0 0" />
+      <geometry>
+        <mesh
+          filename="package://daadbot_desc/meshes/base_claw_link2.STL" />
+      </geometry>
+      <material
+        name="">
+        <color
+          rgba="1 1 1 1" />
+      </material>
+    </visual>
+    <collision>
+      <origin
+        xyz="0 0 0"
+        rpy="0 0 0" />
+      <geometry>
+        <mesh
+          filename="package://daadbot_desc/meshes/base_claw_link2.STL" />
+      </geometry>
+    </collision>
+  </link>
+  <joint
+    name="base_claw_joint2_mimic"
+    type="fixed">
+    <parent
+      link="Link_7" />
+    <child
+      link="dummy_base_claw_joint2_mimic" />
+  </joint>
+  <link name="dummy_base_claw_joint2_mimic"/>
+  <joint
+    name="base_claw_joint2"
+    type="revolute">
+    <origin
+      xyz="0.00500790684313079 0.00524245830200445 0.0685789689082188"
+      rpy="-1.52010273242897 0 0" />
+    <parent
+      link="Link_7" />
+    <child
+      link="base_claw_link2" />
+    <axis
+      xyz="-0.0472460759822792 0.0506152984712578 0.99760007010071" />
     <limit
       lower="0"
@@ -736,4 +896,13 @@
   </link>
   <joint
+    name="claw_joint2_mimic"
+    type="fixed">
+    <parent
+      link="gear2_link" />
+    <child
+      link="dummy_claw_joint2_mimic" />
+  </joint>
+  <link name="dummy_claw_joint2_mimic"/>
+  <joint
     name="claw_joint2"
     type="revolute">
@@ -757,127 +926,3 @@
       offset="0" />
   </joint>
-  <link
-    name="base_claw_link2">
-    <inertial>
-      <origin
-        xyz="0.00030048 -0.015554 -0.00070023"
-        rpy="0 0 0" />
-      <mass
-        value="0.0011042" />
-      <inertia
-        ixx="1.5464E-07"
-        ixy="2.238E-09"
-        ixz="-1.8519E-10"
-        iyy="3.5683E-09"
-        iyz="7.8475E-09"
-        izz="1.5574E-07" />
-    </inertial>
-    <visual>
-      <origin
-        xyz="0 0 0"
-        rpy="0 0 0" />
-      <geometry>
-        <mesh
-          filename="package://daadbot_desc/meshes/base_claw_link2.STL" />
-      </geometry>
-      <material
-        name="">
-        <color
-          rgba="1 1 1 1" />
-      </material>
-    </visual>
-    <collision>
-      <origin
-        xyz="0 0 0"
-        rpy="0 0 0" />
-      <geometry>
-        <mesh
-          filename="package://daadbot_desc/meshes/base_claw_link2.STL" />
-      </geometry>
-    </collision>
-  </link>
-  <joint
-    name="base_claw_joint2"
-    type="revolute">
-    <origin
-      xyz="0.00500790684313079 0.00524245830200445 0.0685789689082188"
-      rpy="-1.52010273242897 0 0" />
-    <parent
-      link="Link_7" />
-    <child
-      link="base_claw_link2" />
-    <axis
-      xyz="-0.0472460759822792 0.0506152984712578 0.99760007010071" />
-    <limit
-      lower="0"
-      upper="0.9"
-      effort="${effort}"
-      velocity="${velocity}" />
-    <mimic
-      joint="gear1_joint"
-      multiplier="-1"
-      offset="0" />
-  </joint>
-  <link
-    name="base_claw_link1">
-    <inertial>
-      <origin
-        xyz="-1.058E-05 -0.015556 -0.00071484"
-        rpy="0 0 0" />
-      <mass
-        value="0.0011042" />
-      <inertia
-        ixx="1.5467E-07"
-        ixy="-7.9881E-10"
-        ixz="-2.9739E-11"
-        iyy="3.5247E-09"
-        iyz="7.7059E-09"
-        izz="1.5576E-07" />
-    </inertial>
-    <visual>
-      <origin
-        xyz="0 0 0"
-        rpy="0 0 0" />
-      <geometry>
-        <mesh
-          filename="package://daadbot_desc/meshes/base_claw_link1.STL" />
-      </geometry>
-      <material
-        name="">
-        <color
-          rgba="1 1 1 1" />
-      </material>
-    </visual>
-    <collision>
-      <origin
-        xyz="0 0 0"
-        rpy="0 0 0" />
-      <geometry>
-        <mesh
-          filename="package://daadbot_desc/meshes/base_claw_link1.STL" />
-      </geometry>
-    </collision>
-  </link>
-  <joint
-    name="base_claw_joint1"
-    type="revolute">
-    <origin
-      xyz="-0.00548036760308535 0.0047463745042049 0.0685789689085226"
-      rpy="-1.52010273242897 0 0" />
-    <parent
-      link="Link_7" />
-    <child
-      link="base_claw_link1" />
-    <axis
-      xyz="0.0472460759822863 -0.0506152984712078 -0.997600070100712" />
-    <limit
-      lower="0"
-      upper="0.9"
-      effort="${effort}"
-      velocity="${velocity}" />
-    <mimic
-      joint="gear1_joint"
-      multiplier="-1"
-      offset="0" />
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