Commit message: Initial Hardware interfcaes without re-purposing for own hardware.

File: src/daadbot_desc/urdf/urdf_oct/daadbot.urdf.xacro (robot description, xacro)
@@ -1,4 +1,6 @@
 <?xml version="1.0" encoding="utf-8"?>
 <robot xmlns:xacro="http://www.ros.org/wiki/xacro" name="daadbot">
+  <!-- Load Simulated or Real Hardware Interfaces -->
+  <xacro:arg name="is_sim" default="true"/>
   <xacro:arg name = "is_ignition" default="true"/>
   <xacro:include filename = "$(find daadbot_desc)/urdf/urdf_oct/daadbot_gazebo.xacro"/>

File: src/daadbot_desc/urdf/urdf_oct/daadbot_ros2_control.xacro (robot description, xacro)
@@ -3,12 +3,59 @@
     <xacro:property name='PI' value='3.141592653589793'/>
     <ros2_control type="system" name="Manipulator">
-        <xacro:if value="$(arg is_ignition)">
+        <!-- ros2_control Gazebo -->
+        <xacro:if value="$(arg is_sim)">
+            <!-- ROS 2 Humble -->
+            <xacro:if value="$(arg is_ignition)">
+                <hardware>
+                    <plugin>ign_ros2_control/IgnitionSystem</plugin>
+                </hardware>
+            </xacro:if>
+            <!-- ROS 2 jazzy -->
+            <xacro:unless value="$(arg is_ignition)">
+                <hardware>
+                    <plugin>gz_ros2_control/GazeboSimSystem</plugin>
+                </hardware>
+            </xacro:unless>
+                <joint name="base_claw_joint1">
+                <param name="mimic">gear1_joint</param>
+                <param name="multiplier">-1</param>
+                <state_interface name="position"/>
+                <state_interface name="velocity"/>
+                <state_interface name="effort"/>
+            </joint>
+            <joint name="claw_joint1">
+                <param name="mimic">base_claw_joint1</param>
+                <param name="multiplier">1</param>
+                <state_interface name="position"/>
+                <state_interface name="velocity"/>
+                <state_interface name="effort"/>
+            </joint>
+            <joint name="gear2_joint">
+                <param name="mimic">gear1_joint</param>
+                <param name="multiplier">-1</param>
+                <state_interface name="position"/>
+                <state_interface name="velocity"/>
+                <state_interface name="effort"/>
+            </joint>
+            <joint name="base_claw_joint2">
+                <param name="mimic">gear1_joint</param>
+                <param name="multiplier">-1</param>
+                <state_interface name="position"/>
+                <state_interface name="velocity"/>
+                <state_interface name="effort"/>
+            </joint>
+            <joint name="claw_joint2">
+                <param name="mimic">base_claw_joint2</param>
+                <param name="multiplier">-1</param>
+                <state_interface name="position"/>
+                <state_interface name="velocity"/>
+                <state_interface name="effort"/>
+            </joint>
+        </xacro:if>
+        <!-- ros2_control Real Robot -->
+        <xacro:unless value="$(arg is_sim)">
             <hardware>
-                <plugin>ign_ros2_control/IgnitionSystem</plugin>
-            </hardware>
-        </xacro:if>
-        <xacro:unless value="$(arg is_ignition)">
-            <hardware>
-                <plugin>gz_ros2_control/GazeboSimSystem</plugin>
+                <plugin>daadbot_controller/DaadbotInterface</plugin>
+                <param name="port">/dev/ttyUSB0</param>
             </hardware>
         </xacro:unless>
@@ -85,39 +132,4 @@
             <state_interface name="effort"/>
         </joint>
-        <joint name="base_claw_joint1">
-            <param name="mimic">gear1_joint</param>
-            <param name="multiplier">-1</param>
-            <state_interface name="position"/>
-            <state_interface name="velocity"/>
-            <state_interface name="effort"/>
-        </joint>
-        <joint name="claw_joint1">
-            <param name="mimic">base_claw_joint1</param>
-            <param name="multiplier">1</param>
-            <state_interface name="position"/>
-            <state_interface name="velocity"/>
-            <state_interface name="effort"/>
-        </joint>
-        <joint name="gear2_joint">
-            <param name="mimic">gear1_joint</param>
-            <param name="multiplier">-1</param>
-            <state_interface name="position"/>
-            <state_interface name="velocity"/>
-            <state_interface name="effort"/>
-        </joint>
-        <joint name="base_claw_joint2">
-            <param name="mimic">gear1_joint</param>
-            <param name="multiplier">-1</param>
-            <state_interface name="position"/>
-            <state_interface name="velocity"/>
-            <state_interface name="effort"/>
-        </joint>
-        <joint name="claw_joint2">
-            <param name="mimic">base_claw_joint2</param>
-            <param name="multiplier">-1</param>
-            <state_interface name="position"/>
-            <state_interface name="velocity"/>
-            <state_interface name="effort"/>
-        </joint>
     </ros2_control>
 </robot>

File: src/daadbot_desc/urdf/urdf_oct_vel/daadbot.urdf.xacro (robot description, xacro)
@@ -1,4 +1,6 @@
 <?xml version="1.0" encoding="utf-8"?>
 <robot xmlns:xacro="http://www.ros.org/wiki/xacro" name="daadbot">
+  <!-- Load Simulated or Real Hardware Interfaces -->
+  <xacro:arg name="is_sim" default="true"/>
   <xacro:arg name = "is_ignition" default="true"/>
   <xacro:include filename = "$(find daadbot_desc)/urdf/urdf_oct_vel/daadbot_gazebo.xacro"/>

File: src/daadbot_desc/urdf/urdf_oct_vel/daadbot_ros2_control.xacro (robot description, xacro)
@@ -3,12 +3,59 @@
     <xacro:property name='PI' value='3.141592653589793'/>
     <ros2_control type="system" name="Manipulator">
-        <xacro:if value="$(arg is_ignition)">
+        <!-- ros2_control Gazebo -->
+        <xacro:if value="$(arg is_sim)">
+            <!-- ROS 2 Humble -->
+            <xacro:if value="$(arg is_ignition)">
+                <hardware>
+                    <plugin>ign_ros2_control/IgnitionSystem</plugin>
+                </hardware>
+            </xacro:if>
+            <!-- ROS 2 jazzy -->
+            <xacro:unless value="$(arg is_ignition)">
+                <hardware>
+                    <plugin>gz_ros2_control/GazeboSimSystem</plugin>
+                </hardware>
+            </xacro:unless>
+                <joint name="base_claw_joint1">
+                <param name="mimic">gear1_joint</param>
+                <param name="multiplier">-1</param>
+                <state_interface name="position"/>
+                <state_interface name="velocity"/>
+                <state_interface name="effort"/>
+            </joint>
+            <joint name="claw_joint1">
+                <param name="mimic">base_claw_joint1</param>
+                <param name="multiplier">1</param>
+                <state_interface name="position"/>
+                <state_interface name="velocity"/>
+                <state_interface name="effort"/>
+            </joint>
+            <joint name="gear2_joint">
+                <param name="mimic">gear1_joint</param>
+                <param name="multiplier">-1</param>
+                <state_interface name="position"/>
+                <state_interface name="velocity"/>
+                <state_interface name="effort"/>
+            </joint>
+            <joint name="base_claw_joint2">
+                <param name="mimic">gear1_joint</param>
+                <param name="multiplier">-1</param>
+                <state_interface name="position"/>
+                <state_interface name="velocity"/>
+                <state_interface name="effort"/>
+            </joint>
+            <joint name="claw_joint2">
+                <param name="mimic">base_claw_joint2</param>
+                <param name="multiplier">-1</param>
+                <state_interface name="position"/>
+                <state_interface name="velocity"/>
+                <state_interface name="effort"/>
+            </joint>
+        </xacro:if>
+        <!-- ros2_control Real Robot -->
+        <xacro:unless value="$(arg is_sim)">
             <hardware>
-                <plugin>ign_ros2_control/IgnitionSystem</plugin>
-            </hardware>
-        </xacro:if>
-        <xacro:unless value="$(arg is_ignition)">
-            <hardware>
-                <plugin>gz_ros2_control/GazeboSimSystem</plugin>
+                <plugin>daadbot_controller/DaadbotInterface</plugin>
+                <param name="port">/dev/ttyUSB0</param>
             </hardware>
         </xacro:unless>
@@ -85,39 +132,4 @@
             <state_interface name="effort"/>
         </joint>
-        <joint name="base_claw_joint1">
-            <param name="mimic">gear1_joint</param>
-            <param name="multiplier">-1</param>
-            <state_interface name="position"/>
-            <state_interface name="velocity"/>
-            <state_interface name="effort"/>
-        </joint>
-        <joint name="claw_joint1">
-            <param name="mimic">base_claw_joint1</param>
-            <param name="multiplier">1</param>
-            <state_interface name="position"/>
-            <state_interface name="velocity"/>
-            <state_interface name="effort"/>
-        </joint>
-        <joint name="gear2_joint">
-            <param name="mimic">gear1_joint</param>
-            <param name="multiplier">-1</param>
-            <state_interface name="position"/>
-            <state_interface name="velocity"/>
-            <state_interface name="effort"/>
-        </joint>
-        <joint name="base_claw_joint2">
-            <param name="mimic">gear1_joint</param>
-            <param name="multiplier">-1</param>
-            <state_interface name="position"/>
-            <state_interface name="velocity"/>
-            <state_interface name="effort"/>
-        </joint>
-        <joint name="claw_joint2">
-            <param name="mimic">base_claw_joint2</param>
-            <param name="multiplier">-1</param>
-            <state_interface name="position"/>
-            <state_interface name="velocity"/>
-            <state_interface name="effort"/>
-        </joint>
     </ros2_control>
 </robot>
