Commit message: Basic Hardware Interface pipeline.

File: src/daadbot_desc/urdf/urdf_table_vel_hw/daadbot.urdf.xacro (robot description, xacro)
@@ -407,5 +407,5 @@
     <limit
       lower="-3.14"
-      upper="3.14"
+      upper="0"
       effort="${effort}"
       velocity="${velocity}" />

File: src/daadbot_desc/urdf/urdf_table_vel_hw/daadbot_ros2_control.xacro (robot description, xacro)
@@ -17,39 +17,4 @@
                 </hardware>
             </xacro:unless>
-                <joint name="base_claw_joint1">
-                <param name="mimic">gear1_joint</param>
-                <param name="multiplier">-1</param>
-                <state_interface name="position"/>
-                <state_interface name="velocity"/>
-                <state_interface name="effort"/>
-            </joint>
-            <joint name="claw_joint1">
-                <param name="mimic">base_claw_joint1</param>
-                <param name="multiplier">1</param>
-                <state_interface name="position"/>
-                <state_interface name="velocity"/>
-                <state_interface name="effort"/>
-            </joint>
-            <joint name="gear2_joint">
-                <param name="mimic">gear1_joint</param>
-                <param name="multiplier">-1</param>
-                <state_interface name="position"/>
-                <state_interface name="velocity"/>
-                <state_interface name="effort"/>
-            </joint>
-            <joint name="base_claw_joint2">
-                <param name="mimic">gear1_joint</param>
-                <param name="multiplier">-1</param>
-                <state_interface name="position"/>
-                <state_interface name="velocity"/>
-                <state_interface name="effort"/>
-            </joint>
-            <joint name="claw_joint2">
-                <param name="mimic">base_claw_joint2</param>
-                <param name="multiplier">-1</param>
-                <state_interface name="position"/>
-                <state_interface name="velocity"/>
-                <state_interface name="effort"/>
-            </joint>
         </xacro:if>
         <!-- ros2_control Real Robot -->
@@ -57,5 +22,5 @@
             <hardware>
                 <plugin>daadbot_controller/DaadbotInterface</plugin>
-                <param name="port">/dev/ttyUSB0</param>
+                <param name="port">/dev/ttyACM0</param>
             </hardware>
         </xacro:unless>
@@ -123,13 +88,4 @@
             <state_interface name="effort"/>
         </joint>
-        <joint name="gear1_joint">
-            <command_interface name="velocity">
-                <param name="min">-30</param>
-                <param name="max">30</param>
-            </command_interface>
-            <state_interface name="position"/>
-            <state_interface name="velocity"/>
-            <state_interface name="effort"/>
-        </joint>
     </ros2_control>
 </robot>

File: src/daadbot_desc/urdf/urdf_table_vel_sim/daadbot.urdf.xacro (robot description, xacro)
@@ -4,7 +4,7 @@
   <xacro:arg name="is_sim" default="true"/>
   <xacro:arg name = "is_ignition" default="true"/>
-  <xacro:include filename = "$(find daadbot_desc)/urdf/urdf_table_vel/daadbot_gazebo.xacro"/>
-  <xacro:include filename = "$(find daadbot_desc)/urdf/urdf_table_vel/daadbot_ros2_control.xacro"/>
-  <xacro:include filename = "$(find daadbot_desc)/urdf/urdf_table_vel/table.xacro"/>
+  <xacro:include filename = "$(find daadbot_desc)/urdf/urdf_table_vel_sim/daadbot_gazebo.xacro"/>
+  <xacro:include filename = "$(find daadbot_desc)/urdf/urdf_table_vel_sim/daadbot_ros2_control.xacro"/>
+  <xacro:include filename = "$(find daadbot_desc)/urdf/urdf_table_vel_sim/table.xacro"/>
   <xacro:property name='PI' value='3.141592653589793'/>
   <xacro:property name='velocity' value='20.0'/>
@@ -12,5 +12,7 @@
   <link name="world"/>
   <!-- Attach the Table to the World -->
-  <joint name="table_joint" type="fixed">
+  <joint
+    name="sim_table_joint"
+    type="fixed">
     <parent link="world"/>
     <child link="table_top"/>
@@ -18,5 +20,7 @@
   </joint>
   <!-- Attach Daadbot to the Table -->
-  <joint name="base_joint" type="fixed">
+  <joint
+    name="sim_base_joint"
+    type="fixed">
     <parent link="table_top"/>
     <child link="base_link"/>
@@ -104,5 +108,5 @@
   </link>
   <joint
-    name="joint_1"
+    name="sim_joint_1"
     type="revolute">
     <origin
@@ -162,5 +166,5 @@
   </link>
   <joint
-    name="joint_2"
+    name="sim_joint_2"
     type="revolute">
     <origin
@@ -220,5 +224,5 @@
   </link>
   <joint
-    name="joint_3"
+    name="sim_joint_3"
     type="revolute">
     <origin
@@ -278,5 +282,5 @@
   </link>
   <joint
-    name="joint_4"
+    name="sim_joint_4"
     type="revolute">
     <origin
@@ -336,5 +340,5 @@
   </link>
   <joint
-    name="joint_5"
+    name="sim_joint_5"
     type="revolute">
     <origin
@@ -394,5 +398,5 @@
   </link>
   <joint
-    name="joint_6"
+    name="sim_joint_6"
     type="revolute">
     <origin
@@ -452,5 +456,5 @@
   </link>
   <joint
-    name="joint_7"
+    name="sim_joint_7"
     type="revolute">
     <origin
@@ -510,5 +514,5 @@
   </link>
   <joint
-    name="endeffector_joint"
+    name="sim_endeffector_joint"
     type="fixed">
     <origin
@@ -563,5 +567,5 @@
   </link>
   <joint
-    name="gear1_joint"
+    name="sim_gear1_joint"
     type="revolute">
     <origin
@@ -621,5 +625,5 @@
   </link>
   <joint
-    name="base_claw_joint1_mimic"
+    name="sim_base_claw_joint1_mimic"
     type="fixed">
     <parent
@@ -630,5 +634,5 @@
   <link name="dummy_base_claw_joint1_mimic"/>
   <joint
-    name="base_claw_joint1"
+    name="sim_base_claw_joint1"
     type="revolute">
     <origin
@@ -692,5 +696,5 @@
   </link>
   <joint
-    name="claw_joint1_mimic"
+    name="sim_claw_joint1_mimic"
     type="fixed">
     <parent
@@ -701,5 +705,5 @@
   <link name="dummy_claw_joint1_mimic"/>
   <joint
-    name="claw_joint1"
+    name="sim_claw_joint1"
     type="revolute">
     <origin
@@ -763,5 +767,5 @@
   </link>
   <joint
-    name="gear2_joint_mimic"
+    name="sim_gear2_joint_mimic"
     type="fixed">
     <parent
@@ -772,5 +776,5 @@
   <link name="dummy_gear2_joint_mimic"/>
   <joint
-    name="gear2_joint"
+    name="sim_gear2_joint"
     type="revolute">
     <origin
@@ -834,5 +838,5 @@
   </link>
   <joint
-    name="base_claw_joint2_mimic"
+    name="sim_base_claw_joint2_mimic"
     type="fixed">
     <parent
@@ -843,5 +847,5 @@
   <link name="dummy_base_claw_joint2_mimic"/>
   <joint
-    name="base_claw_joint2"
+    name="sim_base_claw_joint2"
     type="revolute">
     <origin
@@ -905,5 +909,5 @@
   </link>
   <joint
-    name="claw_joint2_mimic"
+    name="sim_claw_joint2_mimic"
     type="fixed">
     <parent
@@ -914,5 +918,5 @@
   <link name="dummy_claw_joint2_mimic"/>
   <joint
-    name="claw_joint2"
+    name="sim_claw_joint2"
     type="revolute">
     <origin

File: src/daadbot_desc/urdf/urdf_table_vel_sim/daadbot_ros2_control.xacro (robot description, xacro)
@@ -17,5 +17,5 @@
                 </hardware>
             </xacro:unless>
-                <joint name="base_claw_joint1">
+                <joint name="sim_base_claw_joint1">
                 <param name="mimic">gear1_joint</param>
                 <param name="multiplier">-1</param>
@@ -24,5 +24,5 @@
                 <state_interface name="effort"/>
             </joint>
-            <joint name="claw_joint1">
+            <joint name="sim_claw_joint1">
                 <param name="mimic">base_claw_joint1</param>
                 <param name="multiplier">1</param>
@@ -31,5 +31,5 @@
                 <state_interface name="effort"/>
             </joint>
-            <joint name="gear2_joint">
+            <joint name="sim_gear2_joint">
                 <param name="mimic">gear1_joint</param>
                 <param name="multiplier">-1</param>
@@ -38,5 +38,5 @@
                 <state_interface name="effort"/>
             </joint>
-            <joint name="base_claw_joint2">
+            <joint name="sim_base_claw_joint2">
                 <param name="mimic">gear1_joint</param>
                 <param name="multiplier">-1</param>
@@ -45,5 +45,5 @@
                 <state_interface name="effort"/>
             </joint>
-            <joint name="claw_joint2">
+            <joint name="sim_claw_joint2">
                 <param name="mimic">base_claw_joint2</param>
                 <param name="multiplier">-1</param>
@@ -57,8 +57,8 @@
             <hardware>
                 <plugin>daadbot_controller/DaadbotInterface</plugin>
-                <param name="port">/dev/ttyUSB0</param>
+                <param name="port">/dev/ttyACM0</param>
             </hardware>
         </xacro:unless>
-        <joint name="joint_1">
+        <joint name="sim_joint_1">
             <command_interface name="velocity">
                 <param name="min">-30</param>
@@ -69,5 +69,5 @@
             <state_interface name="effort"/>
         </joint>
-        <joint name="joint_2">
+        <joint name="sim_joint_2">
             <command_interface name="velocity">
                 <param name="min">-30</param>
@@ -78,5 +78,5 @@
             <state_interface name="effort"/>
         </joint>
-        <joint name="joint_3">
+        <joint name="sim_joint_3">
             <command_interface name="velocity">
                 <param name="min">-30</param>
@@ -87,5 +87,5 @@
             <state_interface name="effort"/>
         </joint>
-        <joint name="joint_4">
+        <joint name="sim_joint_4">
             <command_interface name="velocity">
                 <param name="min">-30</param>
@@ -96,5 +96,5 @@
             <state_interface name="effort"/>
         </joint>
-        <joint name="joint_5">
+        <joint name="sim_joint_5">
             <command_interface name="velocity">
                 <param name="min">-30</param>
@@ -105,5 +105,5 @@
             <state_interface name="effort"/>
         </joint>
-        <joint name="joint_6">
+        <joint name="sim_joint_6">
             <command_interface name="velocity">
                 <param name="min">-30</param>
@@ -114,5 +114,5 @@
             <state_interface name="effort"/>
         </joint>
-        <joint name="joint_7">
+        <joint name="sim_joint_7">
             <command_interface name="velocity">
                 <param name="min">-30</param>
@@ -123,5 +123,5 @@
             <state_interface name="effort"/>
         </joint>
-        <joint name="gear1_joint">
+        <joint name="sim_gear1_joint">
             <command_interface name="velocity">
                 <param name="min">-30</param>
