Commit message: Setup the new URDF on jazzy with partially tuned effort PID control.

File: src/daadbot_desc/urdf/urdf_new_table_vel/7dof_2motor_small_rod.urdf (robot description, URDF)
Before this commit: robot 7dof_2motor_small_rod, 16 links, 15 joints
Links:
- removed link Link2_2
- removed link Link_2_1
- added link Link_2, mass 2.24401700155026; collision mesh filename=package://daadbot_desc/meshes/Link_2.STL; visual mesh filename=package://daadbot_desc/meshes/Link_2.STL
- added link world
- link Link_1: mass 2.1249 -> 2.34948803406793; geometry collision mesh filename=package://daadbot_desc/meshes/Link_1.STL; visual mesh filename=package://daadbot_desc/meshes/Link_1.STL
- link Link_3: mass 1.3788 -> 1.2718719681393; geometry collision mesh filename=package://daadbot_desc/meshes/Link_3.STL; visual mesh filename=package://daadbot_desc/meshes/Link_3.STL
- link Link_4: mass 3.1743 -> 2.67615775175726; geometry collision mesh filename=package://daadbot_desc/meshes/Link_4.STL; visual mesh filename=package://daadbot_desc/meshes/Link_4.STL
- link Link_5: mass 1.4559 -> 1.29018300951353; geometry collision mesh filename=package://daadbot_desc/meshes/Link_5.STL; visual mesh filename=package://daadbot_desc/meshes/Link_5.STL
- link Link_7: mass 0.13169 -> 0.131686510129341; geometry collision mesh filename=package://daadbot_desc/meshes/Link_7.STL; visual mesh filename=package://daadbot_desc/meshes/Link_7.STL
- link base_claw_link1: mass 0.00110418822863694 -> 0.00110418822863695; geometry collision mesh filename=package://daadbot_desc/meshes/base_claw_link1.STL; visual mesh filename=package://daadbot_desc/meshes/base_claw_link1.STL
- link base_claw_link2: mass 0.00110418822863696 -> 0.00110418822863694; geometry collision mesh filename=package://daadbot_desc/meshes/base_claw_link2.STL; visual mesh filename=package://daadbot_desc/meshes/base_claw_link2.STL
- link base_link: mass 6.9112 -> 6.91122989464636; geometry collision mesh filename=package://daadbot_desc/meshes/base_link.STL; visual mesh filename=package://daadbot_desc/meshes/base_link.STL
- link endeffector: mass 0.15406 -> 0.154057788286255; geometry collision mesh filename=package://daadbot_desc/meshes/endeffector.STL; visual mesh filename=package://daadbot_desc/meshes/endeffector.STL
- link gear1: mass 0.0053 -> 0.00530003886474417; geometry collision mesh filename=package://daadbot_desc/meshes/gear1.STL; visual mesh filename=package://daadbot_desc/meshes/gear1.STL
- link gear1_claw: mass 0.00393743096892516 -> 0.00393743096892517; geometry collision mesh filename=package://daadbot_desc/meshes/gear1_claw.STL; visual mesh filename=package://daadbot_desc/meshes/gear1_claw.STL
- link gear2_claw: mass 0.00393743096892516 -> 0.00393743096892518; geometry collision mesh filename=package://daadbot_desc/meshes/gear2_claw.STL; visual mesh filename=package://daadbot_desc/meshes/gear2_claw.STL
- link gear2_link: mass 0.00576363113945471 -> 0.00576363113945472; geometry collision mesh filename=package://daadbot_desc/meshes/gear2_link.STL; visual mesh filename=package://daadbot_desc/meshes/gear2_link.STL
- link link_6: mass 1.4077 -> 1.30596061805535; geometry collision mesh filename=package://daadbot_desc/meshes/link_6.STL; visual mesh filename=package://daadbot_desc/meshes/link_6.STL
Joints:
- removed joint Joint_1
- removed joint Joint_2_1
- removed joint Joint_3
- removed joint Joint_7
- removed joint joint2_2
- added joint base_joint: type fixed, parent table_top, child base_link, origin xyz=0 0 0 rpy=0 0 0
- added joint joint_1: type revolute, parent base_link, child Link_1, origin xyz=-0.0029638 -0.0015759 0.04796 rpy=0 0 0, axis 0 0 -1, limit lower=0 upper=3.14 effort=22 velocity=12.776
- added joint joint_2: type revolute, parent Link_1, child Link_2, origin xyz=0.0400000000000002 -0.050000000000002 0.114463048454132 rpy=1.5707963267949 0 0, axis 0 0 -1, limit lower=-3.4907 upper=0.5236 effort=22 velocity=12.776
- added joint joint_3: type revolute, parent Link_2, child Link_3, origin xyz=0.234499999999998 0 -0.0495000000000002 rpy=0 1.5707963267949 0, axis 0 0 -1, limit lower=0 upper=3.14 effort=22 velocity=12.776
- added joint joint_7: type revolute, parent link_6, child Link_7, origin xyz=-0.0864999036793499 0 0.0280000000004628 rpy=0 1.5707963267949 0, axis 0 0 -1, limit lower=0 upper=3.14 effort=15 velocity=19.897
- added joint table_joint: type fixed, parent world, child table_top, origin xyz=0 0 0 rpy=0 0 0
- joint base_claw_joint1: axis -1 0 0 -> 0 0 -1; origin xyz=0.0015 -0.00525 -0.066079 rpy=0 0 0 -> xyz=0.00149999999999995 -0.00525000000002329 -0.066078968907985 rpy=0 1.5707963267949 0
- joint base_claw_joint2: axis 1 0 0 -> 0 0 1; origin xyz=0.0015 0.00525 -0.066079 rpy=0 0 0 -> xyz=0.00149999999999995 0.00524999999997672 -0.066078968907985 rpy=0 1.5707963267949 0
- joint claw_joint1: axis 1 0 0 -> 0 0 1; origin xyz=-0.0005 0.0016069 -0.030958 rpy=0 0 0 -> xyz=-0.0309835156221249 -0.00101082129116717 0 rpy=3.14159265358979 0 3.14159265358979
- joint claw_joint2: axis 1 0 0 -> 0 0 1; origin xyz=0.0005 0.0021276 -0.030927 rpy=0 0 0 -> xyz=-0.0309869843208653 0.000898221965043244 -0.00225000000000025 rpy=-3.14159265358979 0 -3.14159265358979
- joint endeffector: origin xyz=0 0 -0.008 rpy=0 0 3.1416 -> xyz=0 0 -0.00799999999954315 rpy=3.14159265357033 0 -3.14159265358979
- joint gear1_joint: axis 1 0 0 -> 0 0 -1; origin xyz=-0.0025 0.0135 -0.037679 rpy=0 0 -3.1416 -> xyz=-0.00375000000000747 -0.013499999998183 0.0376789689084349 rpy=0 1.5707963267949 0
- joint gear2_joint: axis 1 0 0 -> 0 0 -1; origin xyz=-0.0015 -0.0135 -0.037679 rpy=0 0 -3.1416 -> xyz=-0.00149999999999997 0.0134999999992435 0.0376789689087047 rpy=0 1.5707963267949 0
- joint joint_4: origin xyz=-0.0325 0 0.095 rpy=0 1.5708 0 -> xyz=-0.0324999999999996 0 0.0750000000000004 rpy=0 1.5707963267949 0
- joint joint_5: origin xyz=-0.269 0 0.032 rpy=3.1416 1.5708 0 -> xyz=-0.2284999036789 0 0.0330000000000004 rpy=3.14159265358979 1.5707963267949 0; type continuous -> revolute
- joint joint_6: axis 0 0 1 -> 0 0 -1; limit lower=-1.5708 upper=1.5708 effort=15 velocity=19.896753 -> lower=-1.5708 upper=1.5708 effort=15 velocity=19.897; origin xyz=-0.0265 0 0.065 rpy=3.1416 1.5708 0 -> xyz=0.0265000104908596 0 0.0575000000000075 rpy=3.14159265358979 1.5707963267949 0

File: src/daadbot_desc/urdf/urdf_new_table_vel/daadbot.urdf.xacro (robot description, xacro)
@@ -44,5 +44,5 @@
       <geometry>
         <mesh
-          filename="package://daadbot_desc/meshes2/base_link.STL" />
+          filename="package://daadbot_desc/meshes/base_link.STL" />
       </geometry>
       <material
@@ -58,5 +58,5 @@
       <geometry>
         <mesh
-          filename="package://daadbot_desc/meshes2/base_link.STL" />
+          filename="package://daadbot_desc/meshes/base_link.STL" />
       </geometry>
     </collision>
@@ -84,5 +84,5 @@
       <geometry>
         <mesh
-          filename="package://daadbot_desc/meshes2/Link_1.STL" />
+          filename="package://daadbot_desc/meshes/Link_1.STL" />
       </geometry>
       <material
@@ -98,5 +98,5 @@
       <geometry>
         <mesh
-          filename="package://daadbot_desc/meshes2/Link_1.STL" />
+          filename="package://daadbot_desc/meshes/Link_1.STL" />
       </geometry>
     </collision>
@@ -142,5 +142,5 @@
       <geometry>
         <mesh
-          filename="package://daadbot_desc/meshes2/Link_2_1.STL" />
+          filename="package://daadbot_desc/meshes/Link_2_1.STL" />
       </geometry>
       <material
@@ -156,5 +156,5 @@
       <geometry>
         <mesh
-          filename="package://daadbot_desc/meshes2/Link_2_1.STL" />
+          filename="package://daadbot_desc/meshes/Link_2_1.STL" />
       </geometry>
     </collision>
@@ -200,5 +200,5 @@
       <geometry>
         <mesh
-          filename="package://daadbot_desc/meshes2/Link_3.STL" />
+          filename="package://daadbot_desc/meshes/Link_3.STL" />
       </geometry>
       <material
@@ -214,5 +214,5 @@
       <geometry>
         <mesh
-          filename="package://daadbot_desc/meshes2/Link_3.STL" />
+          filename="package://daadbot_desc/meshes/Link_3.STL" />
       </geometry>
     </collision>
@@ -258,5 +258,5 @@
       <geometry>
         <mesh
-          filename="package://daadbot_desc/meshes2/Link_4.STL" />
+          filename="package://daadbot_desc/meshes/Link_4.STL" />
       </geometry>
       <material
@@ -272,5 +272,5 @@
       <geometry>
         <mesh
-          filename="package://daadbot_desc/meshes2/Link_4.STL" />
+          filename="package://daadbot_desc/meshes/Link_4.STL" />
       </geometry>
     </collision>
@@ -316,5 +316,5 @@
       <geometry>
         <mesh
-          filename="package://daadbot_desc/meshes2/Link_5.STL" />
+          filename="package://daadbot_desc/meshes/Link_5.STL" />
       </geometry>
       <material
@@ -330,5 +330,5 @@
       <geometry>
         <mesh
-          filename="package://daadbot_desc/meshes2/Link_5.STL" />
+          filename="package://daadbot_desc/meshes/Link_5.STL" />
       </geometry>
     </collision>
@@ -374,5 +374,5 @@
       <geometry>
         <mesh
-          filename="package://daadbot_desc/meshes2/link_6.STL" />
+          filename="package://daadbot_desc/meshes/link_6.STL" />
       </geometry>
       <material
@@ -388,5 +388,5 @@
       <geometry>
         <mesh
-          filename="package://daadbot_desc/meshes2/link_6.STL" />
+          filename="package://daadbot_desc/meshes/link_6.STL" />
       </geometry>
     </collision>
@@ -432,5 +432,5 @@
       <geometry>
         <mesh
-          filename="package://daadbot_desc/meshes2/Link_7.STL" />
+          filename="package://daadbot_desc/meshes/Link_7.STL" />
       </geometry>
       <material
@@ -446,5 +446,5 @@
       <geometry>
         <mesh
-          filename="package://daadbot_desc/meshes2/Link_7.STL" />
+          filename="package://daadbot_desc/meshes/Link_7.STL" />
       </geometry>
     </collision>
@@ -490,5 +490,5 @@
       <geometry>
         <mesh
-          filename="package://daadbot_desc/meshes2/endeffector.STL" />
+          filename="package://daadbot_desc/meshes/endeffector.STL" />
       </geometry>
       <material
@@ -504,5 +504,5 @@
       <geometry>
         <mesh
-          filename="package://daadbot_desc/meshes2/endeffector.STL" />
+          filename="package://daadbot_desc/meshes/endeffector.STL" />
       </geometry>
     </collision>
@@ -543,5 +543,5 @@
       <geometry>
         <mesh
-          filename="package://daadbot_desc/meshes2/gear1.STL" />
+          filename="package://daadbot_desc/meshes/gear1.STL" />
       </geometry>
       <material
@@ -557,5 +557,5 @@
       <geometry>
         <mesh
-          filename="package://daadbot_desc/meshes2/gear1.STL" />
+          filename="package://daadbot_desc/meshes/gear1.STL" />
       </geometry>
     </collision>
@@ -601,5 +601,5 @@
       <geometry>
         <mesh
-          filename="package://daadbot_desc/meshes2/gear1_claw.STL" />
+          filename="package://daadbot_desc/meshes/gear1_claw.STL" />
       </geometry>
       <material
@@ -615,5 +615,5 @@
       <geometry>
         <mesh
-          filename="package://daadbot_desc/meshes2/gear1_claw.STL" />
+          filename="package://daadbot_desc/meshes/gear1_claw.STL" />
       </geometry>
     </collision>
@@ -663,5 +663,5 @@
       <geometry>
         <mesh
-          filename="package://daadbot_desc/meshes2/gear2_link.STL" />
+          filename="package://daadbot_desc/meshes/gear2_link.STL" />
       </geometry>
       <material
@@ -677,5 +677,5 @@
       <geometry>
         <mesh
-          filename="package://daadbot_desc/meshes2/gear2_link.STL" />
+          filename="package://daadbot_desc/meshes/gear2_link.STL" />
       </geometry>
     </collision>
@@ -725,5 +725,5 @@
       <geometry>
         <mesh
-          filename="package://daadbot_desc/meshes2/gear2_claw.STL" />
+          filename="package://daadbot_desc/meshes/gear2_claw.STL" />
       </geometry>
       <material
@@ -739,5 +739,5 @@
       <geometry>
         <mesh
-          filename="package://daadbot_desc/meshes2/gear2_claw.STL" />
+          filename="package://daadbot_desc/meshes/gear2_claw.STL" />
       </geometry>
     </collision>
@@ -787,5 +787,5 @@
       <geometry>
         <mesh
-          filename="package://daadbot_desc/meshes2/base_claw_link2.STL" />
+          filename="package://daadbot_desc/meshes/base_claw_link2.STL" />
       </geometry>
       <material
@@ -801,5 +801,5 @@
       <geometry>
         <mesh
-          filename="package://daadbot_desc/meshes2/base_claw_link2.STL" />
+          filename="package://daadbot_desc/meshes/base_claw_link2.STL" />
       </geometry>
     </collision>
@@ -849,5 +849,5 @@
       <geometry>
         <mesh
-          filename="package://daadbot_desc/meshes2/base_claw_link1.STL" />
+          filename="package://daadbot_desc/meshes/base_claw_link1.STL" />
       </geometry>
       <material
@@ -863,5 +863,5 @@
       <geometry>
         <mesh
-          filename="package://daadbot_desc/meshes2/base_claw_link1.STL" />
+          filename="package://daadbot_desc/meshes/base_claw_link1.STL" />
       </geometry>
     </collision>
@@ -911,5 +911,5 @@
       <geometry>
         <mesh
-          filename="package://daadbot_desc/meshes2/Link2_2.STL" />
+          filename="package://daadbot_desc/meshes/Link2_2.STL" />
       </geometry>
       <material
@@ -925,5 +925,5 @@
       <geometry>
         <mesh
-          filename="package://daadbot_desc/meshes2/Link2_2.STL" />
+          filename="package://daadbot_desc/meshes/Link2_2.STL" />
       </geometry>
     </collision>
