Commit message: Setup the new URDF on jazzy with partially tuned effort PID control.

File: src/daadbot_desc/urdf/urdf_table_vel/daadbot.urdf.xacro (robot description, xacro)
@@ -1,5 +1,4 @@
 <?xml version="1.0" encoding="utf-8"?>
 <robot xmlns:xacro="http://www.ros.org/wiki/xacro" name="daadbot">
-  <!-- Load Simulated or Real Hardware Interfaces -->
   <xacro:arg name="is_sim" default="true"/>
   <xacro:arg name = "is_ignition" default="true"/>
@@ -9,5 +8,5 @@
   <xacro:property name='PI' value='3.141592653589793'/>
   <xacro:property name='velocity' value='20.0'/>
-  <xacro:property name='effort' value='150.0'/>
+  <xacro:property name='effort' value='200.0'/>
   <link name="world"/>
   <!-- Attach the Table to the World -->
@@ -21,5 +20,5 @@
     <parent link="table_top"/>
     <child link="base_link"/>
-    <origin xyz="0.3 0 0.015" rpy="0 0 0"/> <!-- Adjust position of the robot on the table -->
+    <origin xyz="0.3 0 1.017" rpy="0 0 0"/> <!-- Adjust position of the robot on the table -->
   </joint>
   <link
@@ -27,15 +26,15 @@
     <inertial>
       <origin
-        xyz="0.00049737 0.00026123 0.0072038"
-        rpy="0 0 0" />
-      <mass
-        value="6.9112" />
-      <inertia
-        ixx="0.046617"
-        ixy="0.00010077"
-        ixz="5.1488E-08"
-        iyy="0.046482"
-        iyz="-1.4461E-07"
-        izz="0.092984" />
+        xyz="-0.00246645540256236 -0.00131466478904116 0.00320374562257973"
+        rpy="0 0 0" />
+      <mass
+        value="6.91122989464636" />
+      <inertia
+        ixx="0.0466171750852481"
+        ixy="0.00010076855342015"
+        ixz="5.14819747192778E-08"
+        iyy="0.0464821203083076"
+        iyz="-1.44621889265211E-07"
+        izz="0.0929840869855057" />
     </inertial>
     <visual>
@@ -50,5 +49,5 @@
         name="">
         <color
-          rgba="0.77647 0.75686 0.73725 1" />
+          rgba="0.776470588235294 0.756862745098039 0.737254901960784 1" />
       </material>
     </visual>
@@ -67,15 +66,15 @@
     <inertial>
       <origin
-        xyz="1.4551E-05 -0.0043711 0.069929"
-        rpy="0 0 0" />
-      <mass
-        value="1.4053" />
-      <inertia
-        ixx="0.0017174"
-        ixy="6.6784E-08"
-        ixz="3.5551E-07"
-        iyy="0.002626"
-        iyz="6.0024E-06"
-        izz="0.0017063" />
+        xyz="0.0222146013900772 2.73568109690481E-06 0.0747841784291177"
+        rpy="0 0 0" />
+      <mass
+        value="2.34948803406793" />
+      <inertia
+        ixx="0.00332922517000865"
+        ixy="1.64875308454708E-07"
+        ixz="-0.000433929392474112"
+        iyy="0.00524724735039028"
+        iyz="2.38505609352415E-07"
+        izz="0.00419520671173006" />
     </inertial>
     <visual>
@@ -90,5 +89,5 @@
         name="">
         <color
-          rgba="0 0 0 1" />
+          rgba="0.647058823529412 0.619607843137255 0.588235294117647 1" />
       </material>
     </visual>
@@ -107,6 +106,6 @@
     type="revolute">
     <origin
-      xyz="0 0 0.05"
-      rpy="0 0 3.1416" />
+      xyz="-0.0029638 -0.0015759 0.04796"
+      rpy="0 0 0" />
     <parent
       link="base_link" />
@@ -117,7 +116,7 @@
     <limit
       lower="-0.1"
-      upper="3.145"
+      upper="3.2"
       effort="${effort}"
-      velocity="${velocity}" />
+      velocity="12.776" />
   </joint>
   <link
@@ -125,15 +124,15 @@
     <inertial>
       <origin
-        xyz="-6.5548E-05 0.21409 0.034291"
-        rpy="0 0 0" />
-      <mass
-        value="3.4329" />
-      <inertia
-        ixx="0.0091312"
-        ixy="-2.4753E-06"
-        ixz="8.4256E-07"
-        iyy="0.0057112"
-        iyz="5.0607E-06"
-        izz="0.0099035" />
+        xyz="0.121210588587965 0.000230649813345946 -0.049540637756618"
+        rpy="0 0 0" />
+      <mass
+        value="2.24401700155026" />
+      <inertia
+        ixx="0.00389001580470153"
+        ixy="1.8291659115195E-06"
+        ixz="2.04233321611583E-07"
+        iyy="0.00259728697678572"
+        iyz="3.29392581309982E-08"
+        izz="0.00312685277067708" />
     </inertial>
     <visual>
@@ -148,5 +147,5 @@
         name="">
         <color
-          rgba="1 1 1 1" />
+          rgba="0.898039215686275 0.917647058823529 0.929411764705882 1" />
       </material>
     </visual>
@@ -165,10 +164,126 @@
     type="revolute">
     <origin
-      xyz="0 -0.02999999999948 0.107500000000395"
-      rpy="1.5707963267949 0 -3.14159265358979" />
+      xyz="0.0400000000000002 -0.050000000000002 0.114463048454132"
+      rpy="1.5707963267949 0 0" />
     <parent
       link="Link_1" />
     <child
       link="Link_2" />
+    <axis
+      xyz="0 0 -1" />
+    <limit
+      lower="-3.4907"
+      upper="0.5236"
+      effort="${effort}"
+      velocity="12.776" />
+  </joint>
+  <link
+    name="Link_3">
+    <inertial>
+      <origin
+        xyz="-0.00448997206818821 -2.34751712904213E-05 0.0488571768392556"
+        rpy="0 0 0" />
+      <mass
+        value="1.2718719681393" />
+      <inertia
+        ixx="0.00206983011422612"
+        ixy="9.27500479472452E-08"
+        ixz="3.38378548754623E-06"
+        iyy="0.00129565231901482"
+        iyz="2.88989653562542E-07"
+        izz="0.00156994991003151" />
+    </inertial>
+    <visual>
+      <origin
+        xyz="0 0 0"
+        rpy="0 0 0" />
+      <geometry>
+        <mesh
+          filename="package://daadbot_desc/meshes/Link_3.STL" />
+      </geometry>
+      <material
+        name="">
+        <color
+          rgba="0.898039215686275 0.917647058823529 0.929411764705882 1" />
+      </material>
+    </visual>
+    <collision>
+      <origin
+        xyz="0 0 0"
+        rpy="0 0 0" />
+      <geometry>
+        <mesh
+          filename="package://daadbot_desc/meshes/Link_3.STL" />
+      </geometry>
+    </collision>
+  </link>
+  <joint
+    name="joint_3"
+    type="revolute">
+    <origin
+      xyz="0.234499999999998 0 -0.0495000000000002"
+      rpy="0 1.5707963267949 0" />
+    <parent
+      link="Link_2" />
+    <child
+      link="Link_3" />
+    <axis
+      xyz="0 0 -1" />
+    <limit
+      lower="-0.1"
+      upper="3.2"
+      effort="${effort}"
+      velocity="12.776" />
+  </joint>
+  <link
+    name="Link_4">
+    <inertial>
+      <origin
+        xyz="-0.119169680650385 -0.000128811902195713 0.0378163924527294"
+        rpy="0 0 0" />
+      <mass
+        value="2.67615775175726" />
+      <inertia
+        ixx="0.00308017562479927"
+        ixy="2.47453551729311E-06"
+        ixz="-7.09348932448939E-07"
+        iyy="0.00238129778603005"
+        iyz="-7.47320677385655E-07"
+        izz="0.00293128138362422" />
+    </inertial>
+    <visual>
+      <origin
+        xyz="0 0 0"
+        rpy="0 0 0" />
+      <geometry>
+        <mesh
+          filename="package://daadbot_desc/meshes/Link_4.STL" />
+      </geometry>
+      <material
+        name="">
+        <color
+          rgba="0.898039215686275 0.917647058823529 0.929411764705882 1" />
+      </material>
+    </visual>
+    <collision>
+      <origin
+        xyz="0 0 0"
+        rpy="0 0 0" />
+      <geometry>
+        <mesh
+          filename="package://daadbot_desc/meshes/Link_4.STL" />
+      </geometry>
+    </collision>
+  </link>
+  <joint
+    name="joint_4"
+    type="revolute">
+    <origin
+      xyz="-0.0324999999999996 0 0.0750000000000004"
+      rpy="0 1.5707963267949 0" />
+    <parent
+      link="Link_3" />
+    <child
+      link="Link_4" />
     <axis
       xyz="0 0 -1" />
@@ -177,295 +292,179 @@
       upper="1.9199"
       effort="${effort}"
-      velocity="${velocity}" />
-  </joint>
-  <link
-    name="Link_3">
-    <inertial>
-      <origin
-        xyz="-2.1655E-05 0.0044003 0.0672"
-        rpy="0 0 0" />
-      <mass
-        value="1.3788" />
-      <inertia
-        ixx="0.0016215"
-        ixy="-9.275E-08"
-        ixz="2.8899E-07"
-        iyy="0.0025027"
-        iyz="-5.4475E-06"
-        izz="0.0016785" />
-    </inertial>
-    <visual>
-      <origin
-        xyz="0 0 0"
-        rpy="0 0 0" />
-      <geometry>
-        <mesh
-          filename="package://daadbot_desc/meshes/Link_3.STL" />
-      </geometry>
-      <material
-        name="">
-        <color
-          rgba="0 0 0 1" />
-      </material>
-    </visual>
-    <collision>
-      <origin
-        xyz="0 0 0"
-        rpy="0 0 0" />
-      <geometry>
-        <mesh
-          filename="package://daadbot_desc/meshes/Link_3.STL" />
-      </geometry>
-    </collision>
-  </link>
-  <joint
-    name="joint_3"
-    type="revolute">
-    <origin
-      xyz="0.000359289684152012 0.435033961918617 0.0294474762975983"
-      rpy="1.57079632680726 0 3.14159265358979" />
-    <parent
-      link="Link_2" />
-    <child
-      link="Link_3" />
-    <axis
-      xyz="0 0 -1" />
-    <limit
-      lower="-0.1"
-      upper="3.145"
-      effort="${effort}"
-      velocity="${velocity}" />
-  </joint>
-  <link
-    name="Link_4">
-    <inertial>
-      <origin
-        xyz="0.22054 0.00021752 -0.034312"
-        rpy="0 0 0" />
-      <mass
-        value="3.5515" />
-      <inertia
-        ixx="0.0043885"
-        ixy="2.6288E-06"
-        ixz="-3.6827E-06"
-        iyy="0.0083524"
-        iyz="-3.8569E-06"
-        izz="0.0091315" />
-    </inertial>
-    <visual>
-      <origin
-        xyz="0 0 0"
-        rpy="0 0 0" />
-      <geometry>
-        <mesh
-          filename="package://daadbot_desc/meshes/Link_4.STL" />
-      </geometry>
-      <material
-        name="">
-        <color
-          rgba="1 1 1 1" />
-      </material>
-    </visual>
-    <collision>
-      <origin
-        xyz="0 0 0"
-        rpy="0 0 0" />
-      <geometry>
-        <mesh
-          filename="package://daadbot_desc/meshes/Link_4.STL" />
-      </geometry>
-    </collision>
-  </link>
-  <joint
-    name="joint_4"
-    type="revolute">
-    <origin
-      xyz="0 0.0299999999999995 0.102500000000001"
-      rpy="1.5707963267949 0 3.14159265358979" />
-    <parent
-      link="Link_3" />
-    <child
+      velocity="12.77581" />
+  </joint>
+  <link
+    name="Link_5">
+    <inertial>
+      <origin
+        xyz="0.00685541523757274 3.79292913340323E-05 0.0488580132405974"
+        rpy="0 0 0" />
+      <mass
+        value="1.29018300951353" />
+      <inertia
+        ixx="0.00112308173661534"
+        ixy="1.28316182440177E-06"
+        ixz="-8.91005390036956E-07"
+        iyy="0.000690097277055795"
+        iyz="-3.23958303943101E-07"
+        izz="0.000815216487439054" />
+    </inertial>
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
File: src/daadbot_desc/urdf/urdf_table_vel/table.xacro (robot description, xacro)
@@ -4,5 +4,5 @@
   <link name="table_top">
     <visual>
-      <origin xyz="0 0 0.0"/>
+      <origin xyz="0 0 1.0"/>
       <geometry>
         <box size="1.5 0.8 0.03"/>
@@ -24,11 +24,11 @@
     </inertial>
   </link>
-  <!-- Table Legs -->
+  <!-- Table Legs Macro -->
   <xacro:macro name="table_leg" params="leg_name x y">
     <link name="${leg_name}">
       <visual>
-        <origin xyz="${x} ${y} 0.0"/>
+        <origin xyz="0 0 0.5"/>
         <geometry>
-          <cylinder radius="0.02" length="1"/>
+          <cylinder radius="0.02" length="1.0"/>
         </geometry>
         <material name="">
@@ -37,11 +37,11 @@
       </visual>
       <collision>
-        <origin xyz="${x} ${y} 0.5"/>
+        <origin xyz="0 0 0.5"/>
         <geometry>
-          <cylinder radius="0.02" length="1"/>
+          <cylinder radius="0.02" length="1.0"/>
         </geometry>
       </collision>
       <inertial>
-        <origin xyz="${x} ${y} 0.5"/>
+        <origin xyz="0 0 0.5"/>
         <mass value="1.0"/>
         <inertia ixx="0.01" ixy="0" ixz="0" iyy="0.01" iyz="0" izz="0.01"/>
@@ -51,11 +51,11 @@
       <parent link="table_top"/>
       <child link="${leg_name}"/>
-      <origin xyz="0 0 -0.5"/>
+      <origin xyz="${x} ${y} 0.0"/>
     </joint>
   </xacro:macro>
   <!-- Four Legs -->
-  <xacro:table_leg leg_name="front_left_leg" x="0.68" y="0.38"/>
-  <xacro:table_leg leg_name="front_right_leg" x="0.68" y="-0.38"/>
-  <xacro:table_leg leg_name="back_left_leg" x="-0.68" y="0.38"/>
-  <xacro:table_leg leg_name="back_right_leg" x="-0.68" y="-0.38"/>
+  <xacro:table_leg leg_name="front_left_leg"  x=" 0.68" y=" 0.38"/>
+  <xacro:table_leg leg_name="front_right_leg" x=" 0.68" y="-0.38"/>
+  <xacro:table_leg leg_name="back_left_leg"   x="-0.68" y=" 0.38"/>
+  <xacro:table_leg leg_name="back_right_leg"  x="-0.68" y="-0.38"/>
 </robot>
