Commit message: Changes for new urdf with table.

File: src/daadbot_desc/urdf/urdf_table_vel/daadbot.urdf.xacro (robot description, xacro)
@@ -9,5 +9,5 @@
   <xacro:property name='PI' value='3.141592653589793'/>
   <xacro:property name='velocity' value='20.0'/>
-  <xacro:property name='effort' value='300.0'/>
+  <xacro:property name='effort' value='75.0'/>
   <link name="world"/>
   <!-- Attach the Table to the World -->
@@ -105,5 +105,5 @@
   <joint
     name="joint_1"
-    type="continuous">
+    type="revolute">
     <origin
       xyz="0 0 0.05"
@@ -116,6 +116,6 @@
       xyz="0 0 -1" />
     <limit
-      lower="0"
-      upper="3.14"
+      lower="-0.1"
+      upper="3.145"
       effort="${effort}"
       velocity="${velocity}" />
@@ -221,5 +221,5 @@
   <joint
     name="joint_3"
-    type="continuous">
+    type="revolute">
     <origin
       xyz="0.000359289684152012 0.435033961918617 0.0294474762975983"
@@ -232,6 +232,6 @@
       xyz="0 0 -1" />
     <limit
-      lower="0"
-      upper="3.14"
+      lower="-0.1"
+      upper="3.145"
       effort="${effort}"
       velocity="${velocity}" />
@@ -337,5 +337,5 @@
   <joint
     name="joint_5"
-    type="continuous">
+    type="revolute">
     <origin
       xyz="0.419299903678905 0 -0.0294999999999992"
@@ -348,6 +348,6 @@
       xyz="0 0 -1" />
     <limit
-      lower="0"
-      upper="3.14"
+      lower="-0.1"
+      upper="3.145"
       effort="${effort}"
       velocity="${velocity}" />
@@ -453,5 +453,5 @@
   <joint
     name="joint_7"
-    type="continuous">
+    type="revolute">
     <origin
       xyz="0 -0.0909999036788988 -0.0244999999999991"
@@ -464,6 +464,6 @@
       xyz="0 0 -1" />
     <limit
-      lower="0"
-      upper="3.14"
+      lower="-0.1"
+      upper="3.145"
       effort="${effort}"
       velocity="${velocity}" />

File: src/daadbot_desc/urdf/urdf_table_vel/daadbot_ros2_control.xacro (robot description, xacro)
@@ -22,4 +22,5 @@
                 <state_interface name="position"/>
                 <state_interface name="velocity"/>
+                <state_interface name="effort"/>
             </joint>
             <joint name="claw_joint1">
@@ -28,4 +29,5 @@
                 <state_interface name="position"/>
                 <state_interface name="velocity"/>
+                <state_interface name="effort"/>
             </joint>
             <joint name="gear2_joint">
@@ -34,4 +36,5 @@
                 <state_interface name="position"/>
                 <state_interface name="velocity"/>
+                <state_interface name="effort"/>
             </joint>
             <joint name="base_claw_joint2">
@@ -40,4 +43,5 @@
                 <state_interface name="position"/>
                 <state_interface name="velocity"/>
+                <state_interface name="effort"/>
             </joint>
             <joint name="claw_joint2">
@@ -46,4 +50,5 @@
                 <state_interface name="position"/>
                 <state_interface name="velocity"/>
+                <state_interface name="effort"/>
             </joint>
         </xacro:if>
@@ -62,4 +67,5 @@
             <state_interface name="position"/>
             <state_interface name="velocity"/>
+            <state_interface name="effort"/>
         </joint>
         <joint name="joint_2">
@@ -70,4 +76,5 @@
             <state_interface name="position"/>
             <state_interface name="velocity"/>
+            <state_interface name="effort"/>
         </joint>
         <joint name="joint_3">
@@ -78,4 +85,5 @@
             <state_interface name="position"/>
             <state_interface name="velocity"/>
+            <state_interface name="effort"/>
         </joint>
         <joint name="joint_4">
@@ -86,4 +94,5 @@
             <state_interface name="position"/>
             <state_interface name="velocity"/>
+            <state_interface name="effort"/>
         </joint>
         <joint name="joint_5">
@@ -94,4 +103,5 @@
             <state_interface name="position"/>
             <state_interface name="velocity"/>
+            <state_interface name="effort"/>
         </joint>
         <joint name="joint_6">
@@ -102,4 +112,5 @@
             <state_interface name="position"/>
             <state_interface name="velocity"/>
+            <state_interface name="effort"/>
         </joint>
         <joint name="joint_7">
@@ -110,4 +121,5 @@
             <state_interface name="position"/>
             <state_interface name="velocity"/>
+            <state_interface name="effort"/>
         </joint>
         <joint name="gear1_joint">
@@ -118,4 +130,5 @@
             <state_interface name="position"/>
             <state_interface name="velocity"/>
+            <state_interface name="effort"/>
         </joint>
     </ros2_control>

Commit message: Basic hardware-interface code changes for getting state and command interfaces.
Also, a trajectory plotting file to visualize the generated trajectory from moveit.

File: src/daadbot_desc/urdf/urdf_table_vel/daadbot.urdf.xacro (robot description, xacro)
@@ -9,5 +9,5 @@
   <xacro:property name='PI' value='3.141592653589793'/>
   <xacro:property name='velocity' value='20.0'/>
-  <xacro:property name='effort' value='75.0'/>
+  <xacro:property name='effort' value='150.0'/>
   <link name="world"/>
   <!-- Attach the Table to the World -->

File: src/daadbot_desc/urdf/urdf_table_vel/daadbot_ros2_control.xacro (robot description, xacro)
@@ -57,5 +57,5 @@
             <hardware>
                 <plugin>daadbot_controller/DaadbotInterface</plugin>
-                <param name="port">/dev/ttyUSB0</param>
+                <param name="port">/dev/ttyACM0</param>
             </hardware>
         </xacro:unless>

Commit message: The new hw interface for only the base motor. Previous one with last 3 motors in daadbot_interface_last.cpp.
Changed the URDF to have downward link 7 (joint 6 = -90) (Present in urdf_table_vel_n)

File: src/daadbot_desc/urdf/urdf_table_vel/daadbot.urdf.xacro (robot description, xacro)
@@ -20,5 +20,5 @@
     <parent link="table_top"/>
     <child link="base_link"/>
-    <origin xyz="0.3 0 1.017" rpy="0 0 0"/> <!-- Adjust position of the robot on the table -->
+    <origin xyz="0.30 0 1.017" rpy="0 0 0"/> <!-- Adjust position of the robot on the table -->
   </joint>
   <link

File: src/daadbot_desc/urdf/urdf_table_vel_n/daadbot.urdf.xacro (robot description, xacro)
@@ -5,14 +5,20 @@
   <xacro:include filename = "$(find daadbot_desc)/urdf/urdf_table_vel/daadbot_gazebo.xacro"/>
   <xacro:include filename = "$(find daadbot_desc)/urdf/urdf_table_vel/daadbot_ros2_control.xacro"/>
+  <xacro:include filename = "$(find daadbot_desc)/urdf/urdf_table_vel/table.xacro"/>
   <xacro:property name='PI' value='3.141592653589793'/>
   <xacro:property name='velocity' value='20.0'/>
-  <xacro:property name='effort' value='300.0'/>
+  <xacro:property name='effort' value='200.0'/>
   <link name="world"/>
   <!-- Attach the Table to the World -->
+  <joint name="table_joint" type="fixed">
+    <parent link="world"/>
+    <child link="table_top"/>
+    <origin xyz="0 0 0" rpy="0 0 0"/> <!-- Adjust height of table -->
+  </joint>
   <!-- Attach Daadbot to the Table -->
   <joint name="base_joint" type="fixed">
-    <parent link="world"/>
+    <parent link="table_top"/>
     <child link="base_link"/>
-    <origin xyz="0.0 0.0 0.0" rpy="0 0 0"/> <!-- Adjust position of the robot on the table -->
+    <origin xyz="0.30 0 1.017" rpy="0 0 0"/> <!-- Adjust position of the robot on the table -->
   </joint>
   <link
@@ -390,6 +396,6 @@
     type="revolute">
     <origin
-      xyz="0.0265000104908596 0 0.0575000000000075"
-      rpy="3.14159265358979 1.5707963267949 0" />
+      xyz="-0.0265000104908596 0 0.0575000000000075"
+      rpy="-1.57 0 -1.57" />
     <parent
       link="Link_5" />

Commit message: Added camera rgb and depth image to launch file - cam_bot.launch.py

File: src/daadbot_desc/urdf/urdf_table_vel/daadbot.urdf.xacro (robot description, xacro)
@@ -141,10 +141,10 @@
         value="2.24401700155026" />
       <inertia
-        ixx="0.00389001580470153"
-        ixy="1.8291659115195E-06"
-        ixz="2.04233321611583E-07"
-        iyy="0.00259728697678572"
-        iyz="3.29392581309982E-08"
-        izz="0.00312685277067708" />
+        ixx="0.00250860362"
+        ixy="-1.95804141e-05"
+        ixz="1.06350024e-06"
+        iyy="0.00852523380"
+        iyz="4.22077320e-07"
+        izz="0.00807927033" />
     </inertial>
     <visual>
@@ -205,4 +205,11 @@
     </sensor>
   </gazebo>
+  <!-- <gazebo>
+   <plugin
+        name="gz::sim::systems::ApplyJointForce"
+        filename="ignition-gazebo-apply-joint-force-system">
+      <joint_name>joint_2</joint_name>
+    </plugin>
+  </gazebo> -->
   <link
     name="Link_3">
@@ -263,4 +270,16 @@
       velocity="12.776" />
   </joint>
+  <gazebo reference="joint_3">
+    <sensor name="tcp_fts_sensor_joint_3" type="force_torque">
+      <always_on>true</always_on>
+      <update_rate>1000</update_rate>
+      <visualize>true</visualize>
+      <force_torque>
+        <frame>child</frame>
+        <measure_direction>child_to_parent</measure_direction>
+      </force_torque>
+      <pose>0 0 0 0 0 0</pose>
+    </sensor>
+  </gazebo>
   <link
     name="Link_4">
@@ -321,4 +340,16 @@
       velocity="12.77581" />
   </joint>
+  <gazebo reference="joint_4">
+    <sensor name="tcp_fts_sensor_joint_4" type="force_torque">
+      <always_on>true</always_on>
+      <update_rate>1000</update_rate>
+      <visualize>true</visualize>
+      <force_torque>
+        <frame>child</frame>
+        <measure_direction>child_to_parent</measure_direction>
+      </force_torque>
+      <pose>0 0 0 0 0 0</pose>
+    </sensor>
+  </gazebo>
   <link
     name="Link_5">
@@ -379,4 +410,16 @@
       velocity="19.896753" />
   </joint>
+  <gazebo reference="joint_5">
+    <sensor name="tcp_fts_sensor_joint_5" type="force_torque">
+      <always_on>true</always_on>
+      <update_rate>1000</update_rate>
+      <visualize>true</visualize>
+      <force_torque>
+        <frame>child</frame>
+        <measure_direction>child_to_parent</measure_direction>
+      </force_torque>
+      <pose>0 0 0 0 0 0</pose>
+    </sensor>
+  </gazebo>
   <link
     name="Link_6">
@@ -437,4 +480,16 @@
       velocity="19.897" />
   </joint>
+  <gazebo reference="joint_6">
+    <sensor name="tcp_fts_sensor_joint_6" type="force_torque">
+      <always_on>true</always_on>
+      <update_rate>1000</update_rate>
+      <visualize>true</visualize>
+      <force_torque>
+        <frame>child</frame>
+        <measure_direction>child_to_parent</measure_direction>
+      </force_torque>
+      <pose>0 0 0 0 0 0</pose>
+    </sensor>
+  </gazebo>
   <link
     name="Link_7">
@@ -495,4 +550,16 @@
       velocity="19.897" />
   </joint>
+  <gazebo reference="joint_7">
+    <sensor name="tcp_fts_sensor_joint_7" type="force_torque">
+      <always_on>true</always_on>
+      <update_rate>1000</update_rate>
+      <visualize>true</visualize>
+      <force_torque>
+        <frame>child</frame>
+        <measure_direction>child_to_parent</measure_direction>
+      </force_torque>
+      <pose>0 0 0 0 0 0</pose>
+    </sensor>
+  </gazebo>
   <link
     name="endeffector">

File: src/daadbot_desc/urdf/urdf_table_vel/daadbot_gazebo.xacro (robot description, xacro)
@@ -3,5 +3,5 @@
     <gazebo>
         <xacro:if value="$(arg is_ignition)">
-            <plugin filename="ign_ros2_control-system" name="ign_ros2_control::IgnitionROS2ControlPlugin">
+            <plugin filename="gz_ros2_control-system" name="gz_ros2_control::GazeboSimROS2ControlPlugin">
                 <parameters>$(find daadbot_controller)/config/vel_trajectory_controller.yaml</parameters>
             </plugin>

File: src/daadbot_desc/urdf/urdf_table_vel/daadbot_ros2_control.xacro (robot description, xacro)
@@ -8,5 +8,5 @@
             <xacro:if value="$(arg is_ignition)">
                 <hardware>
-                    <plugin>ign_ros2_control/IgnitionSystem</plugin>
+                    <plugin>gz_ros2_control/GazeboSimSystem</plugin>
                 </hardware>
             </xacro:if>

File: src/daadbot_desc/urdf/urdf_table_vel/gdaadbot.urdf.xacro (robot description, xacro)
@@ -26,5 +26,5 @@
             <origin xyz="0.002964 0.001576 0.004000" rpy="-3.141593 3.141593 -3.141593" />
             <geometry>
-                <mesh filename="package://daadbot_desc/meshes/base_link.STL" />
+                <mesh filename="/home/maryammahmood/xdaadbot_ws/src/daadbot_desc/dae/final_7dof_assemblyLatest2_base_link_visual_vis_1.dae" />
             </geometry>
         </collision>
@@ -32,5 +32,5 @@
             <origin xyz="0.002964 0.001576 0.004000" rpy="-3.141593 3.141593 -3.141593" />
             <geometry>
-                <mesh filename="package://daadbot_desc/meshes/base_link.STL" />
+                <mesh filename="/home/maryammahmood/xdaadbot_ws/src/daadbot_desc/dae/final_7dof_assemblyLatest2_base_link_visual_vis_1.dae" />
             </geometry>
             <material name="">

File: src/daadbot_desc/urdf/urdf_table_vel/table.xacro (robot description, xacro)
@@ -24,4 +24,22 @@
     </inertial>
   </link>
+  <!-- Make table static in Gazebo and improve contact -->
+  <gazebo reference="table_top">
+    <static>true</static>
+    <surface>
+      <contact>
+        <ode>
+          <kp>100000.0</kp>
+          <kd>1000.0</kd>
+        </ode>
+      </contact>
+      <friction>
+        <ode>
+          <mu>1.0</mu>
+          <mu2>1.0</mu2>
+        </ode>
+      </friction>
+    </surface>
+  </gazebo>
   <!-- Table Legs Macro -->
   <xacro:macro name="table_leg" params="leg_name x y">
