Commit message: some minimal working of dual interface.

File: src/daadbot_desc/urdf/urdf_table_vel/daadbot.urdf.xacro (robot description, xacro)
@@ -115,5 +115,5 @@
       xyz="0 0 -1" />
     <limit
-      lower="-0.1"
+      lower="-3.1"
       upper="3.2"
       effort="${effort}"
@@ -165,5 +165,5 @@
     <origin
       xyz="0.0400000000000002 -0.050000000000002 0.114463048454132"
-      rpy="1.5707963267949 0 0" />
+      rpy="1.5707963267949 -1.83 0" />
     <parent
       link="Link_1" />
@@ -174,5 +174,5 @@
     <limit
       lower="-3.4907"
-      upper="0.5236"
+      upper="3.5236"
       effort="${effort}"
       velocity="12.776" />
@@ -231,8 +231,8 @@
       xyz="0 0 -1" />
     <limit
-      lower="-0.1"
+      lower="-3.1"
       upper="3.2"
       effort="${effort}"
-      velocity="12.776" />
+      velocity="1.0" />
   </joint>
   <link
@@ -281,5 +281,5 @@
     <origin
       xyz="-0.0324999999999996 0 0.0750000000000004"
-      rpy="0 1.5707963267949 0" />
+      rpy="-1.57 0 -1.57" />
     <parent
       link="Link_3" />
@@ -287,10 +287,10 @@
       link="Link_4" />
     <axis
-      xyz="0 0 -1" />
+      xyz="0 0 1" />
     <limit
       lower="-1.9199"
       upper="1.9199"
       effort="${effort}"
-      velocity="12.77581" />
+      velocity="1.0" />
   </joint>
   <link
@@ -339,5 +339,5 @@
     <origin
       xyz="-0.2284999036789 0 0.0330000000000004"
-      rpy="3.14159265358979 1.5707963267949 0" />
+      rpy="3.14159265358979 -1.5707963267949 3.14159" />
     <parent
       link="Link_4" />
@@ -397,5 +397,5 @@
     <origin
       xyz="-0.0265000104908596 0 0.0575000000000075"
-      rpy="-1.57 0 -1.57" />
+      rpy="-1.57 0.2967 -1.57" />
     <parent
       link="Link_5" />
@@ -461,5 +461,5 @@
       link="Link_7" />
     <axis
-      xyz="0 0 -1" />
+      xyz="0 0 1" />
     <limit
       lower="-0.1"

File: src/daadbot_desc/urdf/urdf_table_vel/daadbot_ros2_control.xacro (robot description, xacro)
@@ -1,135 +1,122 @@
 <?xml version="1.0" encoding="utf-8"?>
 <robot xmlns:xacro="http://www.ros.org/wiki/xacro" name="daadbot">
-    <xacro:property name='PI' value='3.141592653589793'/>
-    <ros2_control type="system" name="Manipulator">
-        <!-- ros2_control Gazebo -->
-        <xacro:if value="$(arg is_sim)">
-            <!-- ROS 2 Humble -->
-            <xacro:if value="$(arg is_ignition)">
-                <hardware>
-                    <plugin>ign_ros2_control/IgnitionSystem</plugin>
-                </hardware>
-            </xacro:if>
-            <!-- ROS 2 jazzy -->
-            <xacro:unless value="$(arg is_ignition)">
-                <hardware>
-                    <plugin>gz_ros2_control/GazeboSimSystem</plugin>
-                </hardware>
-            </xacro:unless>
-                <joint name="base_claw_joint1">
-                <param name="mimic">gear1_joint</param>
-                <param name="multiplier">-1</param>
-                <state_interface name="position"/>
-                <state_interface name="velocity"/>
-                <state_interface name="effort"/>
-            </joint>
-            <joint name="claw_joint1">
-                <param name="mimic">base_claw_joint1</param>
-                <param name="multiplier">1</param>
-                <state_interface name="position"/>
-                <state_interface name="velocity"/>
-                <state_interface name="effort"/>
-            </joint>
-            <joint name="gear2_joint">
-                <param name="mimic">gear1_joint</param>
-                <param name="multiplier">-1</param>
-                <state_interface name="position"/>
-                <state_interface name="velocity"/>
-                <state_interface name="effort"/>
-            </joint>
-            <joint name="base_claw_joint2">
-                <param name="mimic">gear1_joint</param>
-                <param name="multiplier">-1</param>
-                <state_interface name="position"/>
-                <state_interface name="velocity"/>
-                <state_interface name="effort"/>
-            </joint>
-            <joint name="claw_joint2">
-                <param name="mimic">base_claw_joint2</param>
-                <param name="multiplier">-1</param>
-                <state_interface name="position"/>
-                <state_interface name="velocity"/>
-                <state_interface name="effort"/>
-            </joint>
-        </xacro:if>
-        <!-- ros2_control Real Robot -->
-        <xacro:unless value="$(arg is_sim)">
-            <hardware>
-                <plugin>daadbot_controller/DaadbotInterface</plugin>
-                <param name="port">/dev/ttyUSB0</param>
-            </hardware>
-        </xacro:unless>
-        <joint name="joint_1">
-            <command_interface name="velocity">
-                <param name="min">-30</param>
-                <param name="max">30</param>
-            </command_interface>
-            <state_interface name="position"/>
-            <state_interface name="velocity"/>
-            <state_interface name="effort"/>
-        </joint>
-        <joint name="joint_2">
-            <command_interface name="velocity">
-                <param name="min">-30</param>
-                <param name="max">30</param>
-            </command_interface>
-            <state_interface name="position"/>
-            <state_interface name="velocity"/>
-            <state_interface name="effort"/>
-        </joint>
-        <joint name="joint_3">
-            <command_interface name="velocity">
-                <param name="min">-30</param>
-                <param name="max">30</param>
-            </command_interface>
-            <state_interface name="position"/>
-            <state_interface name="velocity"/>
-            <state_interface name="effort"/>
-        </joint>
-        <joint name="joint_4">
-            <command_interface name="velocity">
-                <param name="min">-30</param>
-                <param name="max">30</param>
-            </command_interface>
-            <state_interface name="position"/>
-            <state_interface name="velocity"/>
-            <state_interface name="effort"/>
-        </joint>
-        <joint name="joint_5">
-            <command_interface name="velocity">
-                <param name="min">-30</param>
-                <param name="max">30</param>
-            </command_interface>
-            <state_interface name="position"/>
-            <state_interface name="velocity"/>
-            <state_interface name="effort"/>
-        </joint>
-        <joint name="joint_6">
-            <command_interface name="velocity">
-                <param name="min">-30</param>
-                <param name="max">30</param>
-            </command_interface>
-            <state_interface name="position"/>
-            <state_interface name="velocity"/>
-            <state_interface name="effort"/>
-        </joint>
-        <joint name="joint_7">
-            <command_interface name="velocity">
-                <param name="min">-30</param>
-                <param name="max">30</param>
-            </command_interface>
-            <state_interface name="position"/>
-            <state_interface name="velocity"/>
-            <state_interface name="effort"/>
-        </joint>
-        <joint name="gear1_joint">
-            <command_interface name="velocity">
-                <param name="min">-30</param>
-                <param name="max">30</param>
-            </command_interface>
-            <state_interface name="position"/>
-            <state_interface name="velocity"/>
-            <state_interface name="effort"/>
-        </joint>
+  <xacro:property name="PI" value="3.141592653589793"/>
+  <!-- Simulation setup -->
+  <xacro:if value="$(arg is_sim)">
+    <xacro:if value="$(arg is_ignition)">
+      <ros2_control type="system" name="SimSystem">
+        <hardware>
+          <plugin>ign_ros2_control/IgnitionSystem</plugin>
+        </hardware>
+      </ros2_control>
+    </xacro:if>
+    <xacro:unless value="$(arg is_ignition)">
+      <ros2_control type="system" name="SimSystem">
+        <hardware>
+          <plugin>gz_ros2_control/GazeboSimSystem</plugin>
+        </hardware>
+      </ros2_control>
+    </xacro:unless>
+    <!-- Mimic joints for simulation -->
+    <joint name="base_claw_joint1">
+      <param name="mimic">gear1_joint</param>
+      <param name="multiplier">-1</param>
+      <state_interface name="position"/>
+      <state_interface name="velocity"/>
+      <state_interface name="effort"/>
+    </joint>
+    <joint name="claw_joint1">
+      <param name="mimic">base_claw_joint1</param>
+      <param name="multiplier">1</param>
+      <state_interface name="position"/>
+      <state_interface name="velocity"/>
+      <state_interface name="effort"/>
+    </joint>
+    <joint name="gear2_joint">
+      <param name="mimic">gear1_joint</param>
+      <param name="multiplier">-1</param>
+      <state_interface name="position"/>
+      <state_interface name="velocity"/>
+      <state_interface name="effort"/>
+    </joint>
+    <joint name="base_claw_joint2">
+      <param name="mimic">gear1_joint</param>
+      <param name="multiplier">-1</param>
+      <state_interface name="position"/>
+      <state_interface name="velocity"/>
+      <state_interface name="effort"/>
+    </joint>
+    <joint name="claw_joint2">
+      <param name="mimic">base_claw_joint2</param>
+      <param name="multiplier">-1</param>
+      <state_interface name="position"/>
+      <state_interface name="velocity"/>
+      <state_interface name="effort"/>
+    </joint>
+  </xacro:if>
+  <!-- Real hardware configuration -->
+  <xacro:unless value="$(arg is_sim)">
+    <!-- ========== Serial Interface (ESP, USB0) ========== -->
+    <ros2_control type="system" name="SerialManipulator">
+      <hardware>
+        <plugin>daadbot_controller/DaadbotInterface</plugin>
+        <param name="port">/dev/ttyUSB0</param>
+      </hardware>
+      <joint name="joint_5">
+        <command_interface name="velocity"/>
+        <state_interface name="position"/>
+        <state_interface name="velocity"/>
+        <state_interface name="effort"/>
+      </joint>
+      <joint name="joint_6">
+        <command_interface name="velocity"/>
+        <state_interface name="position"/>
+        <state_interface name="velocity"/>
+        <state_interface name="effort"/>
+      </joint>
+      <joint name="joint_7">
+        <command_interface name="velocity"/>
+        <state_interface name="position"/>
+        <state_interface name="velocity"/>
+        <state_interface name="effort"/>
+      </joint>
+      <joint name="gear1_joint">
+        <command_interface name="velocity"/>
+        <state_interface name="position"/>
+        <state_interface name="velocity"/>
+        <state_interface name="effort"/>
+      </joint>
     </ros2_control>
+    <!-- ========== CAN Interface (SocketCAN) ========== -->
+    <ros2_control type="system" name="CANManipulator">
+      <hardware>
+        <plugin>daadbot_controller/CANInterface</plugin>
+        <param name="can_interface">can0</param>
+      </hardware>
+      <joint name="joint_1">
+        <command_interface name="velocity"/>
+        <state_interface name="position"/>
+        <state_interface name="velocity"/>
+        <state_interface name="effort"/>
+      </joint>
+      <joint name="joint_2">
+        <command_interface name="velocity"/>
+        <state_interface name="position"/>
+        <state_interface name="velocity"/>
+        <state_interface name="effort"/>
+      </joint>
+      <joint name="joint_3">
+        <command_interface name="velocity"/>
+        <state_interface name="position"/>
+        <state_interface name="velocity"/>
+        <state_interface name="effort"/>
+      </joint>
+      <joint name="joint_4">
+        <command_interface name="velocity"/>
+        <state_interface name="position"/>
+        <state_interface name="velocity"/>
+        <state_interface name="effort"/>
+      </joint>
+    </ros2_control>
+  </xacro:unless>
 </robot>

Commit message: changes to handpose for new urdf (non-inverted)

File: src/daadbot_desc/urdf/urdf_table_vel/daadbot.urdf.xacro (robot description, xacro)
@@ -16,9 +16,23 @@
     <origin xyz="0 0 0" rpy="0 0 0"/> <!-- Adjust height of table -->
   </joint>
+  <link name="camera_link">
+    <visual>
+      <geometry>
+        <box size="0.05 0.05 0.05"/>
+      </geometry>
+      <material name=""/>
+    </visual>
+  </link>
+  <!-- Fixed joint from base_link to camera_link -->
+  <joint name="camera_joint" type="fixed">
+    <parent link="table_top"/>  <!-- Replace with actual mount link -->
+    <child link="camera_link"/>
+    <origin xyz="1.5 0.0 1.27" rpy="0 0 0"/>
+  </joint>
   <!-- Attach Daadbot to the Table -->
   <joint name="base_joint" type="fixed">
     <parent link="table_top"/>
     <child link="base_link"/>
-    <origin xyz="0.30 0 1.017" rpy="0 0 0"/> <!-- Adjust position of the robot on the table -->
+    <origin xyz="0.55 0 1.017" rpy="0 0 0"/> <!-- Adjust position of the robot on the table -->
   </joint>
   <link
@@ -119,4 +133,10 @@
       effort="${effort}"
       velocity="12.776" />
+  </joint>
+  <link name="daadbot/joint_1/tcp_fts_sensor_joint_1"/>
+  <joint name="tcp_fts_joint_1" type="fixed">
+    <parent link="base_link"/>
+    <child link="daadbot/joint_1/tcp_fts_sensor_joint_1"/>
+    <origin xyz="-0.0029638 -0.0015759 0.04796" rpy="0 0 0"/>
   </joint>
   <gazebo reference="joint_1">
@@ -193,9 +213,15 @@
     </sensor>
   </joint>
+  <link name="daadbot/joint_2/tcp_fts_sensor_joint_2"/>
+  <joint name="tcp_fts_joint_2" type="fixed">
+    <parent link="Link_1"/>
+    <child link="daadbot/joint_2/tcp_fts_sensor_joint_2"/>
+    <origin xyz="0.04 -0.05 0.114463048454132" rpy="1.5707963267949 0 0"/>
+  </joint>
   <gazebo reference="joint_2">
     <sensor name="tcp_fts_sensor_joint_2" type="force_torque">
       <always_on>true</always_on>
-      <update_rate>1000</update_rate>
-      <visualize>true</visualize>
+      <update_rate>100</update_rate>
+      <visualize>false</visualize>
       <force_torque>
         <frame>child</frame>
@@ -270,4 +296,10 @@
       velocity="12.776" />
   </joint>
+  <link name="daadbot/joint_3/tcp_fts_sensor_joint_3"/>
+  <joint name="tcp_fts_joint_3" type="fixed">
+    <parent link="Link_2"/>
+    <child link="daadbot/joint_3/tcp_fts_sensor_joint_3"/>
+    <origin xyz="0.234499999999998 0 -0.04950000000000022" rpy="0 1.5707963267949 0"/>
+  </joint>
   <gazebo reference="joint_3">
     <sensor name="tcp_fts_sensor_joint_3" type="force_torque">
@@ -340,4 +372,10 @@
       velocity="12.77581" />
   </joint>
+  <link name="daadbot/joint_4/tcp_fts_sensor_joint_4"/>
+  <joint name="tcp_fts_joint_4" type="fixed">
+    <parent link="Link_3"/>
+    <child link="daadbot/joint_4/tcp_fts_sensor_joint_4"/>
+    <origin xyz="-0.0324999999999996 0 0.0750000000000004" rpy="0 1.5707963267949 0"/>
+  </joint>
   <gazebo reference="joint_4">
     <sensor name="tcp_fts_sensor_joint_4" type="force_torque">
@@ -410,4 +448,10 @@
       velocity="19.896753" />
   </joint>
+  <link name="daadbot/joint_5/tcp_fts_sensor_joint_5"/>
+  <joint name="tcp_fts_joint_5" type="fixed">
+    <parent link="Link_4"/>
+    <child link="daadbot/joint_5/tcp_fts_sensor_joint_5"/>
+    <origin xyz="-0.2284999036789 0 0.0330000000000004" rpy="3.14159265358979 1.5707963267949 0"/>
+  </joint>
   <gazebo reference="joint_5">
     <sensor name="tcp_fts_sensor_joint_5" type="force_torque">
@@ -480,4 +524,10 @@
       velocity="19.897" />
   </joint>
+  <link name="daadbot/joint_6/tcp_fts_sensor_joint_6"/>
+  <joint name="tcp_fts_joint_6" type="fixed">
+    <parent link="Link_5"/>
+    <child link="daadbot/joint_6/tcp_fts_sensor_joint_6"/>
+    <origin xyz="-0.0265000104908596 0 0.0575000000000075" rpy="-1.57 0 -1.57"/>
+  </joint>
   <gazebo reference="joint_6">
     <sensor name="tcp_fts_sensor_joint_6" type="force_torque">
@@ -550,4 +600,10 @@
       velocity="19.897" />
   </joint>
+  <link name="daadbot/joint_7/tcp_fts_sensor_joint_7"/>
+  <joint name="tcp_fts_joint_7" type="fixed">
+    <parent link="Link_6"/>
+    <child link="daadbot/joint_7/tcp_fts_sensor_joint_7"/>
+    <origin xyz="-0.0864999036793499 0 0.0280000000004628" rpy="0 1.5707963267949 0"/>
+  </joint>
   <gazebo reference="joint_7">
     <sensor name="tcp_fts_sensor_joint_7" type="force_torque">
