Commit message: created a torque trajectory based controller and setup (URDF, moveit) for the data collection

File: src/daadbot_desc/urdf/urdf_inverted/daadbot_org.urdf.xacro (robot description, xacro)
@@ -5,6 +5,5 @@
   <xacro:include filename = "$(find daadbot_desc)/urdf/urdf_inverted/daadbot_gazebo.xacro"/>
   <xacro:include filename = "$(find daadbot_desc)/urdf/urdf_inverted/daadbot_ros2_control.xacro"/>
-  <xacro:include filename = "$(find daadbot_desc)/urdf/urdf_inverted/table_inv.xacro"/>
-  <!-- <xacro:include filename = "$(find daadbot_desc)/urdf/urdf_inverted/lab_table.xacro"/> -->
+  <xacro:include filename = "$(find daadbot_desc)/urdf/urdf_inverted/lab_table.xacro"/>
   <xacro:property name='PI' value='3.141592653589793'/>
   <xacro:property name='velocity' value='20.0'/>
@@ -21,5 +20,5 @@
     <parent link="table_top"/>
     <child link="base_link"/>
-    <origin xyz="0.000 0.0 1.285" rpy="0 3.14 0"/> <!-- Adjust position of the robot on the table -->
+    <origin xyz="0.005 0.1725 1.24" rpy="0 3.14 1.57"/> <!-- Adjust position of the robot on the table -->
     <!-- For inverted - I have changed rpy to 0 3.14 0 from rpy = 0 0 0 -->
   </joint>

File: src/daadbot_desc/urdf/urdf_inverted_torque/daadbot.urdf.xacro (robot description, xacro)
@@ -3,11 +3,11 @@
   <xacro:arg name="is_sim" default="true"/>
   <xacro:arg name = "is_ignition" default="true"/>
-  <xacro:include filename = "$(find daadbot_desc)/urdf/urdf_inverted/daadbot_gazebo.xacro"/>
-  <xacro:include filename = "$(find daadbot_desc)/urdf/urdf_inverted/daadbot_ros2_control.xacro"/>
-  <xacro:include filename = "$(find daadbot_desc)/urdf/urdf_inverted/table_inv.xacro"/>
-  <!-- <xacro:include filename = "$(find daadbot_desc)/urdf/urdf_inverted/lab_table.xacro"/> -->
+  <xacro:include filename = "$(find daadbot_desc)/urdf/urdf_inverted_torque/daadbot_gazebo.xacro"/>
+  <xacro:include filename = "$(find daadbot_desc)/urdf/urdf_inverted_torque/daadbot_ros2_control.xacro"/>
+  <xacro:include filename = "$(find daadbot_desc)/urdf/urdf_inverted_torque/table_inv.xacro"/>
+  <!-- <xacro:include filename = "$(find daadbot_desc)/urdf/urdf_inverted_torque/lab_table.xacro"/> -->
   <xacro:property name='PI' value='3.141592653589793'/>
   <xacro:property name='velocity' value='20.0'/>
-  <xacro:property name='effort' value='200.0'/>
+  <xacro:property name='effort' value='180.0'/>
   <link name="world"/>
   <!-- Attach the Table to the World -->
@@ -117,5 +117,5 @@
       xyz="0 0 -1" />
     <limit
-      lower="-0.1"
+      lower="-3.2"
       upper="3.2"
       effort="${effort}"
@@ -247,5 +247,5 @@
       xyz="0 0 -1" />
     <limit
-      lower="-0.1"
+      lower="-3.2"
       upper="3.2"
       effort="${effort}"
@@ -305,6 +305,6 @@
       xyz="0 0 -1" />
     <limit
-      lower="-1.9199"
-      upper="1.9199"
+      lower="-3.14"
+      upper="3.14"
       effort="${effort}"
       velocity="12.77581" />
@@ -363,5 +363,5 @@
       xyz="0 0 -1" />
     <limit
-      lower="-0.1"
+      lower="-3.2"
       upper="3.4"
       effort="15"
@@ -421,6 +421,6 @@
       xyz="0 0 -1" />
     <limit
-      lower="-1.5708"
-      upper="1.5708"
+      lower="-3.2"
+      upper="3.2"
       effort="15"
       velocity="19.897" />
@@ -479,6 +479,6 @@
       xyz="0 0 -1" />
     <limit
-      lower="0"
-      upper="3.14"
+      lower="-3.2"
+      upper="3.2"
       effort="15"
       velocity="19.897" />

File: src/daadbot_desc/urdf/urdf_inverted_torque/daadbot_org.urdf.xacro (robot description, xacro)
@@ -3,8 +3,7 @@
   <xacro:arg name="is_sim" default="true"/>
   <xacro:arg name = "is_ignition" default="true"/>
-  <xacro:include filename = "$(find daadbot_desc)/urdf/urdf_inverted/daadbot_gazebo.xacro"/>
-  <xacro:include filename = "$(find daadbot_desc)/urdf/urdf_inverted/daadbot_ros2_control.xacro"/>
-  <xacro:include filename = "$(find daadbot_desc)/urdf/urdf_inverted/table_inv.xacro"/>
-  <!-- <xacro:include filename = "$(find daadbot_desc)/urdf/urdf_inverted/lab_table.xacro"/> -->
+  <xacro:include filename = "$(find daadbot_desc)/urdf/urdf_inverted_torque/daadbot_gazebo.xacro"/>
+  <xacro:include filename = "$(find daadbot_desc)/urdf/urdf_inverted_torque/daadbot_ros2_control.xacro"/>
+  <xacro:include filename = "$(find daadbot_desc)/urdf/urdf_inverted_torque/lab_table.xacro"/>
   <xacro:property name='PI' value='3.141592653589793'/>
   <xacro:property name='velocity' value='20.0'/>
@@ -21,5 +20,5 @@
     <parent link="table_top"/>
     <child link="base_link"/>
-    <origin xyz="0.000 0.0 1.285" rpy="0 3.14 0"/> <!-- Adjust position of the robot on the table -->
+    <origin xyz="0.005 0.1725 1.24" rpy="0 3.14 1.57"/> <!-- Adjust position of the robot on the table -->
     <!-- For inverted - I have changed rpy to 0 3.14 0 from rpy = 0 0 0 -->
   </joint>
