Commit message: Scripts for ctc, data collection, dynamics training, and IK along with CLF implementations.

File: src/daadbot_desc/urdf/urdf_inverted_torque/daadbot_noisy.urdf (robot description, URDF)
Before this commit: robot daadbot, 18 links, 17 joints
Links:
- link Link_1: mass 2.297775 -> 2.290365
- link Link_2: mass 2.228958 -> 2.366636
- link Link_3: mass 1.286272 -> 1.295515
- link Link_4: mass 2.567141 -> 2.516984
- link Link_5: mass 1.288714 -> 1.280752
- link Link_6: mass 1.227256 -> 1.226669
- link Link_7: mass 0.128342 -> 0.128382
- link base_claw_link1: mass 0.001138 -> 0.001137
- link base_link: mass 7.234380 -> 7.080898
- link endeffector: mass 0.155172 -> 0.155248
- link gear1: mass 0.004866 -> 0.004867
- link gear1_claw: mass 0.004035 -> 0.004034
- link table_link1: mass 0.000993 -> 0.000985
- link table_top: mass 48.095098 -> 48.599542

Commit message: Re-doing the CLF-CBF. A trajectory viewing in Rviz2

File: src/daadbot_desc/urdf/urdf_inverted_torque/daadbot_noisy.urdf (robot description, URDF)
Before this commit: robot daadbot, 18 links, 17 joints
Links:
- link Link_1: mass 2.290365 -> 2.241993
- link Link_2: mass 2.366636 -> 2.083467
- link Link_3: mass 1.295515 -> 1.240171
- link Link_4: mass 2.516984 -> 2.579729
- link Link_5: mass 1.280752 -> 1.282287
- link Link_6: mass 1.226669 -> 1.227973
- link Link_7: mass 0.128382 -> 0.128236
- link base_claw_link1: mass 0.001137 -> 0.001138
- link base_claw_link2: mass 0.001096 -> 0.001097
- link base_link: mass 7.080898 -> 7.335173
- link endeffector: mass 0.155248 -> 0.155180
- link gear1: mass 0.004867 -> 0.004863
- link gear1_claw: mass 0.004034 -> 0.004037
- link gear2_claw: mass 0.003904 -> 0.003905
- link gear2_link: mass 0.006158 -> 0.006161
- link table_link1: mass 0.000985 -> 0.000991
- link table_top: mass 48.599542 -> 48.289999
