Commit message: URDF with lab table as commented line in new urdf

File: src/daadbot_desc/urdf/urdf_inverted_torque/daadbot.urdf.xacro (robot description, xacro)
@@ -22,4 +22,5 @@
     <child link="base_link"/>
     <origin xyz="0.000 0.0 1.285" rpy="0 3.14 0"/> <!-- Adjust position of the robot on the table -->
+    <!-- <origin xyz="0.005 0.1725 1.24" rpy="0 3.14 1.57"/>-->
     <!-- For inverted - I have changed rpy to 0 3.14 0 from rpy = 0 0 0 -->
   </joint>

Commit message: Got the 2-motors based link 1 replaced with gear-box integrated link1

File: src/daadbot_desc/urdf/urdf_inverted_torque/daadbot.urdf.xacro (robot description, xacro)
@@ -6,8 +6,8 @@
   <xacro:include filename = "$(find daadbot_desc)/urdf/urdf_inverted_torque/daadbot_ros2_control.xacro"/>
   <xacro:include filename = "$(find daadbot_desc)/urdf/urdf_inverted_torque/table_inv.xacro"/>
-  <!-- <xacro:include filename = "$(find daadbot_desc)/urdf/urdf_inverted_torque/lab_table.xacro"/> -->
+  <!-- <xacro:include filename = "$(find daadbot_desc)/urdf/urdf_inverted/lab_table.xacro"/> -->
   <xacro:property name='PI' value='3.141592653589793'/>
   <xacro:property name='velocity' value='20.0'/>
-  <xacro:property name='effort' value='180.0'/>
+  <xacro:property name='effort' value='35.0'/>
   <link name="world"/>
   <!-- Attach the Table to the World -->
@@ -122,4 +122,5 @@
       effort="${effort}"
       velocity="12.776" />
+      <dynamics damping="0.3" friction="0.0"/>
   </joint>
   <gazebo reference="joint_1">
@@ -191,4 +192,5 @@
       effort="${effort}"
       velocity="12.776" />
+      <dynamics damping="0.3" friction="0.0"/>
     <sensor name="force_torque" type="force_torque">
           <update_rate>30</update_rate>
@@ -252,4 +254,5 @@
       effort="${effort}"
       velocity="12.776" />
+      <dynamics damping="0.3" friction="0.0"/>
   </joint>
   <link
@@ -310,4 +313,5 @@
       effort="${effort}"
       velocity="12.77581" />
+      <dynamics damping="0.3" friction="0.0"/>
   </joint>
   <link
@@ -367,5 +371,6 @@
       upper="3.4"
       effort="15"
-      velocity="19.896753" />
+      velocity="9.896753" />
+      <dynamics damping="0.3" friction="0.0"/>
   </joint>
   <link
@@ -425,5 +430,6 @@
       upper="3.2"
       effort="15"
-      velocity="19.897" />
+      velocity="9.897" />
+      <dynamics damping="0.3" friction="0.0"/>
   </joint>
   <link
@@ -483,5 +489,6 @@
       upper="3.2"
       effort="15"
-      velocity="19.897" />
+      velocity="0.0" />
+      <dynamics damping="0.3" friction="0.0"/>
   </joint>
   <link
@@ -594,5 +601,6 @@
       upper="0"
       effort="5"
-      velocity="10" />
+      velocity="0.0" />
+      <dynamics damping="0.3" friction="0.0"/>
   </joint>
   <link

File: src/daadbot_desc/urdf/urdf_inverted_torque/daadbot_gazebo.xacro (robot description, xacro)
@@ -1,5 +1,5 @@
 <?xml version="1.0" encoding="utf-8"?>
 <robot xmlns:xacro="http://www.ros.org/wiki/xacro" name="daadbot">
-    <gazebo>
+    <!-- <gazebo>
         <xacro:if value="$(arg is_ignition)">
             <plugin filename="ign_ros2_control-system" name="ign_ros2_control::IgnitionROS2ControlPlugin">
@@ -12,4 +12,16 @@
             </plugin>
         </xacro:unless>
+    </gazebo> -->
+    <gazebo>
+        <xacro:if value="$(arg is_ignition)">
+            <plugin filename="ign_ros2_control-system" name="ign_ros2_control::IgnitionROS2ControlPlugin">
+                <parameters>$(find daadbot_controller)/config/effort_command_controller.yaml</parameters>
+            </plugin>
+        </xacro:if>
+        <xacro:unless value="$(arg is_ignition)">
+            <plugin filename="gz_ros2_control-system" name="gz_ros2_control::GazeboSimROS2ControlPlugin">
+                <parameters>$(find daadbot_controller)/config/effort_command_controller.yaml</parameters>
+            </plugin>
+        </xacro:unless>
     </gazebo>
 </robot>

File: src/daadbot_desc/urdf/urdf_inverted_torque/daadbot_ros2_control.xacro (robot description, xacro)
@@ -62,6 +62,6 @@
         <joint name="joint_1">
             <command_interface name="effort">
-                <param name="min">-180</param>
-                <param name="max">180</param>
+                <param name="min">-18</param>
+                <param name="max">18</param>
             </command_interface>
             <state_interface name="position"/>
@@ -71,6 +71,6 @@
         <joint name="joint_2">
             <command_interface name="effort">
-                <param name="min">-180</param>
-                <param name="max">180</param>
+                <param name="min">-45</param>
+                <param name="max">45</param>
             </command_interface>
             <state_interface name="position"/>
@@ -80,6 +80,6 @@
         <joint name="joint_3">
             <command_interface name="effort">
-                <param name="min">-180</param>
-                <param name="max">180</param>
+                <param name="min">-18</param>
+                <param name="max">18</param>
             </command_interface>
             <state_interface name="position"/>
@@ -89,6 +89,6 @@
         <joint name="joint_4">
             <command_interface name="effort">
-                <param name="min">-180</param>
-                <param name="max">180</param>
+                <param name="min">-18</param>
+                <param name="max">18</param>
             </command_interface>
             <state_interface name="position"/>
@@ -98,6 +98,6 @@
         <joint name="joint_5">
             <command_interface name="effort">
-                <param name="min">-180</param>
-                <param name="max">180</param>
+                <param name="min">-5</param>
+                <param name="max">5</param>
             </command_interface>
             <state_interface name="position"/>
@@ -107,6 +107,6 @@
         <joint name="joint_6">
             <command_interface name="effort">
-                <param name="min">-180</param>
-                <param name="max">180</param>
+                <param name="min">-5</param>
+                <param name="max">5</param>
             </command_interface>
             <state_interface name="position"/>
@@ -116,6 +116,6 @@
         <joint name="joint_7">
             <command_interface name="effort">
-                <param name="min">-180</param>
-                <param name="max">180</param>
+                <param name="min">-5</param>
+                <param name="max">5</param>
             </command_interface>
             <state_interface name="position"/>

Commit message: Added the transparency argument for the transparent top launch to be able to view x-y plane top view of robot (CBF barrier)

File: src/daadbot_desc/urdf/urdf_inverted_torque/daadbot.urdf.xacro (robot description, xacro)
@@ -3,4 +3,7 @@
   <xacro:arg name="is_sim" default="true"/>
   <xacro:arg name = "is_ignition" default="true"/>
+  <xacro:arg name="transparent_top" default="false"/>
+  <xacro:property name="table_alpha" value="${'0.15' if '$(arg transparent_top)' == 'true' else '1.0'}"/>
+  <xacro:property name="base_link_alpha" value="${'0.27' if '$(arg transparent_top)' == 'true' else '1.0'}"/>
   <xacro:include filename = "$(find daadbot_desc)/urdf/urdf_inverted_torque/daadbot_gazebo.xacro"/>
   <xacro:include filename = "$(find daadbot_desc)/urdf/urdf_inverted_torque/daadbot_ros2_control.xacro"/>
@@ -52,5 +55,5 @@
         name="">
         <color
-          rgba= "1 1 1 1" />
+          rgba= "1 1 1 ${base_link_alpha}" />
       </material>
     </visual>

File: src/daadbot_desc/urdf/urdf_inverted_torque/table_inv.xacro (robot description, xacro)
@@ -16,5 +16,5 @@
       </geometry>
       <material name="grey_base">
-        <color rgba="0.81 0.81 0.63 1" />
+        <color rgba="0.81 0.81 0.63 ${table_alpha}" />
       </material>
     </visual>
