Commit message: modified urdf for different joint limits

File: src/daadbot_desc/urdf/urdf_inverted_torque/daadbot.urdf (robot description, URDF)
Before this commit: robot daadbot, 18 links, 17 joints
Links:
- link Link_1: geometry collision mesh filename=package://daadbot_desc/meshes/Link_1.STL; visual mesh filename=package://daadbot_desc/meshes/Link_1.STL
- link Link_2: geometry collision mesh filename=package://daadbot_desc/meshes/Link_2.STL; visual mesh filename=package://daadbot_desc/meshes/Link_2.STL
- link Link_3: geometry collision mesh filename=package://daadbot_desc/meshes/Link_3.STL; visual mesh filename=package://daadbot_desc/meshes/Link_3.STL
- link Link_4: geometry collision mesh filename=package://daadbot_desc/meshes/Link_4.STL; visual mesh filename=package://daadbot_desc/meshes/Link_4.STL
- link Link_5: geometry collision mesh filename=package://daadbot_desc/meshes/Link_5.STL; visual mesh filename=package://daadbot_desc/meshes/Link_5.STL
- link Link_6: geometry collision mesh filename=package://daadbot_desc/meshes/link_6.STL; visual mesh filename=package://daadbot_desc/meshes/link_6.STL
- link Link_7: geometry collision mesh filename=package://daadbot_desc/meshes/Link_7.STL; visual mesh filename=package://daadbot_desc/meshes/Link_7.STL
- link base_claw_link1: geometry collision mesh filename=package://daadbot_desc/meshes/base_claw_link1.STL; visual mesh filename=package://daadbot_desc/meshes/base_claw_link1.STL
- link base_claw_link2: geometry collision mesh filename=package://daadbot_desc/meshes/base_claw_link2.STL; visual mesh filename=package://daadbot_desc/meshes/base_claw_link2.STL
- link base_link: geometry collision mesh filename=package://daadbot_desc/meshes/base_link.STL; visual mesh filename=package://daadbot_desc/meshes/base_link.STL
- link endeffector: geometry collision mesh filename=package://daadbot_desc/meshes/endeffector.STL; visual mesh filename=package://daadbot_desc/meshes/endeffector.STL
- link gear1: geometry collision mesh filename=package://daadbot_desc/meshes/gear1.STL; visual mesh filename=package://daadbot_desc/meshes/gear1.STL
- link gear1_claw: geometry collision mesh filename=package://daadbot_desc/meshes/gear1_claw.STL; visual mesh filename=package://daadbot_desc/meshes/gear1_claw.STL
- link gear2_claw: geometry collision mesh filename=package://daadbot_desc/meshes/gear2_claw.STL; visual mesh filename=package://daadbot_desc/meshes/gear2_claw.STL
- link gear2_link: geometry collision mesh filename=package://daadbot_desc/meshes/gear2_link.STL; visual mesh filename=package://daadbot_desc/meshes/gear2_link.STL
Joints:
- joint joint_1: limit lower=-3.2 upper=3.2 effort=35.0 velocity=12.776 -> lower=-3.2 upper=3.2 effort=40.0 velocity=1.2
- joint joint_2: limit lower=-3.4907 upper=3.5236 effort=35.0 velocity=12.776 -> lower=-1.745 upper=1.745 effort=40.0 velocity=1.2
- joint joint_3: limit lower=-3.2 upper=3.2 effort=35.0 velocity=12.776 -> lower=-3.2 upper=3.2 effort=40.0 velocity=1.2
- joint joint_4: limit lower=-3.14 upper=3.14 effort=35.0 velocity=12.77581 -> lower=-1.745 upper=1.745 effort=40.0 velocity=1.2
- joint joint_5: limit lower=-3.2 upper=3.4 effort=15 velocity=9.896753 -> lower=-3.2 upper=3.4 effort=15 velocity=1.2
- joint joint_6: limit lower=-3.2 upper=3.2 effort=15 velocity=9.897 -> lower=-1.57 upper=1.57 effort=15 velocity=1.2
- joint joint_7: limit lower=-3.2 upper=3.2 effort=15 velocity=0.0 -> lower=-3.2 upper=3.2 effort=15 velocity=1.2

File: src/daadbot_desc/urdf/urdf_inverted_torque/daadbot.urdf.xacro (robot description, xacro)
@@ -8,6 +8,6 @@
   <!-- <xacro:include filename = "$(find daadbot_desc)/urdf/urdf_inverted/lab_table.xacro"/> -->
   <xacro:property name='PI' value='3.141592653589793'/>
-  <xacro:property name='velocity' value='20.0'/>
-  <xacro:property name='effort' value='35.0'/>
+  <xacro:property name='velocity' value='1.2'/>
+  <xacro:property name='effort' value='40.0'/>
   <link name="world"/>
   <!-- Attach the Table to the World -->
@@ -121,5 +121,5 @@
       upper="3.2"
       effort="${effort}"
-      velocity="12.776" />
+      velocity="${velocity}" />
       <dynamics damping="0.3" friction="0.0"/>
   </joint>
@@ -188,8 +188,8 @@
       xyz="0 0 -1" />
     <limit
-      lower="-3.4907"
-      upper="3.5236"
+      lower="-1.745"
+      upper="1.745"
       effort="${effort}"
-      velocity="12.776" />
+      velocity="${velocity}" />
       <dynamics damping="0.3" friction="0.0"/>
     <sensor name="force_torque" type="force_torque">
@@ -253,5 +253,5 @@
       upper="3.2"
       effort="${effort}"
-      velocity="12.776" />
+      velocity="${velocity}" />
       <dynamics damping="0.3" friction="0.0"/>
   </joint>
@@ -309,8 +309,8 @@
       xyz="0 0 -1" />
     <limit
-      lower="-3.14"
-      upper="3.14"
+      lower="-1.745"
+      upper="1.745"
       effort="${effort}"
-      velocity="12.77581" />
+      velocity="${velocity}" />
       <dynamics damping="0.3" friction="0.0"/>
   </joint>
@@ -371,5 +371,5 @@
       upper="3.4"
       effort="15"
-      velocity="9.896753" />
+      velocity="${velocity}" />
       <dynamics damping="0.3" friction="0.0"/>
   </joint>
@@ -427,8 +427,8 @@
       xyz="0 0 -1" />
     <limit
-      lower="-3.2"
-      upper="3.2"
+      lower="-1.57"
+      upper="1.57"
       effort="15"
-      velocity="9.897" />
+      velocity="${velocity}" />
       <dynamics damping="0.3" friction="0.0"/>
   </joint>
@@ -489,5 +489,5 @@
       upper="3.2"
       effort="15"
-      velocity="0.0" />
+      velocity="${velocity}" />
       <dynamics damping="0.3" friction="0.0"/>
   </joint>

File: src/daadbot_desc/urdf/urdf_inverted_torque/daadbot_ros2_control.xacro (robot description, xacro)
@@ -71,6 +71,6 @@
         <joint name="joint_2">
             <command_interface name="effort">
-                <param name="min">-45</param>
-                <param name="max">45</param>
+                <param name="min">-39</param>
+                <param name="max">39</param>
             </command_interface>
             <state_interface name="position"/>

Commit message: Pinocchio physics based main node + Qunatile calculation

File: src/daadbot_desc/urdf/urdf_inverted_torque/daadbot.urdf (robot description, URDF)
Before this commit: robot daadbot, 18 links, 17 joints
Links:
- link Link_1: mass 2.297775 -> 2.34948803406793
- link Link_2: mass 2.228958 -> 2.24401700155026
- link Link_3: mass 1.286272 -> 1.2718719681393
- link Link_4: mass 2.567141 -> 2.67615775175726
- link Link_5: mass 1.288714 -> 1.29018300951353
- link Link_6: mass 1.227256 -> 1.30596061805535
- link Link_7: mass 0.128342 -> 0.131686510129341
- link base_claw_link1: mass 0.001138 -> 0.00110418822863695
- link base_claw_link2: mass 0.001096 -> 0.00110418822863694
- link base_link: mass 7.234380 -> 6.91122989464636
- link endeffector: mass 0.155172 -> 0.154057788286255
- link gear1: mass 0.004866 -> 0.00530003886474417
- link gear1_claw: mass 0.004035 -> 0.00393743096892517
- link gear2_claw: mass 0.003904 -> 0.00393743096892518
- link gear2_link: mass 0.006158 -> 0.00576363113945472
- link table_link1: mass 0.000993 -> 0.001
- link table_top: mass 48.095098 -> 50.0
Joints:
- joint joint_3: limit lower=-3.2 upper=3.2 effort=40.0 velocity=1.2 -> lower=-7.0 upper=7.0 effort=40.0 velocity=1.2

File: src/daadbot_desc/urdf/urdf_inverted_torque/daadbot.urdf.xacro (robot description, xacro)
@@ -253,6 +253,6 @@
       xyz="0 0 -1" />
     <limit
-      lower="-3.2"
-      upper="3.2"
+      lower="-7.0"
+      upper="7.0"
       effort="${effort}"
       velocity="${velocity}" />

File: src/daadbot_desc/urdf/urdf_inverted_torque/daadbot_noisy2.urdf (robot description, URDF)
Before this commit: robot daadbot, 18 links, 17 joints
Links:
- link Link_1: mass 1.708949 -> 2.305098
- link Link_2: mass 2.831867 -> 2.205944
- link Link_3: mass 0.496334 -> 1.322597
- link Link_4: mass 0.759921 -> 2.687092
- link Link_5: mass 1.525283 -> 1.285506
- link Link_6: mass 1.747265 -> 1.305233
- link Link_7: mass 0.112604 -> 0.131722
- link base_claw_link1: mass 0.001138 -> 0.001105
- link base_claw_link2: mass 0.001096 -> 0.001104
- link base_link: mass 7.234380 -> 6.779607
- link endeffector: mass 0.155172 -> 0.154058
- link gear1: mass 0.004866 -> 0.005305
- link gear1_claw: mass 0.004035 -> 0.003941
- link gear2_claw: mass 0.003904 -> 0.003937
- link gear2_link: mass 0.006158 -> 0.005766
- link table_link1: mass 0.000993 -> 0.000989
- link table_top: mass 48.095098 -> 49.604667

File: src/daadbot_desc/urdf/urdf_inverted_torque/daadbot_noisy_.urdf (robot description, URDF)
Before this commit: robot daadbot, 18 links, 17 joints
Links:
- link Link_1: mass 1.708949 -> 1.840594
- link Link_2: mass 2.831867 -> 1.880291
- link Link_3: mass 0.496334 -> 1.521430
- link Link_4: mass 0.759921 -> 2.508624
- link Link_5: mass 1.525283 -> 1.321643
- link Link_6: mass 1.747265 -> 1.527108
- link Link_7: mass 0.112604 -> 0.132694
- link base_claw_link1: mass 0.001138 -> 0.00110418822863695
- link base_claw_link2: mass 0.001096 -> 0.00110418822863694
- link base_link: mass 7.234380 -> 6.91122989464636
- link endeffector: mass 0.155172 -> 0.154057788286255
- link gear1: mass 0.004866 -> 0.00530003886474417
- link gear1_claw: mass 0.004035 -> 0.00393743096892517
- link gear2_claw: mass 0.003904 -> 0.00393743096892518
- link gear2_link: mass 0.006158 -> 0.00576363113945472
- link table_link1: mass 0.000993 -> 0.001
- link table_top: mass 48.095098 -> 50.0
