Commit message: Reprposed main node, qp_solver, trajectory generator, and clf, cbf for the 2_link. Basic setup nut not perfect working one

File: src/daadbot_desc/urdf/2_link_urdf/2link_robot.urdf.xacro (robot description, xacro)
@@ -27,5 +27,31 @@
         <visual>
             <geometry>
-                <box size="1 .05 .05"/>
+                <box size="0.75 .11 .11"/>
+            </geometry>
+            <origin rpy="0 0 0" xyz="0.375 0 0"/>
+            <material name="black"/>
+        </visual>
+        <collision>
+            <geometry>
+                <box size="0.75 .11 .11"/>
+            </geometry>
+            <origin rpy="0 0 0" xyz="0.375 0 0"/>
+        </collision>
+        <inertial>
+            <origin rpy="0 0 0" xyz="0.375 0 0"/>
+            <mass value="2.0"/>
+            <inertia ixx="0.001" ixy="0" ixz="0" iyy="0.08" iyz="0" izz="0.08"/>
+        </inertial>
+    </link>
+    <joint name="baseHinge" type="revolute">
+        <axis rpy="0 0 0" xyz="0 0 1"/>
+        <limit effort="50.0" velocity="1.0" lower="-3.14159" upper="3.14159"/>
+        <parent link="base"/>
+        <child link="arm1"/>
+    </joint>
+    <link name="arm2">
+        <visual>
+            <geometry>
+                <box size="1 .06 .06"/>
             </geometry>
             <origin rpy="0 0 0" xyz="0.5 0 0"/>
@@ -34,5 +60,5 @@
         <collision>
             <geometry>
-                <box size="1 .05 .05"/>
+                <box size="1 .06 .06"/>
             </geometry>
             <origin rpy="0 0 0" xyz="0.5 0 0"/>
@@ -40,38 +66,14 @@
         <inertial>
             <origin rpy="0 0 0" xyz="0.5 0 0"/>
-            <mass value="1.0"/>
+            <mass value="1.5"/>
             <inertia ixx="0.001" ixy="0" ixz="0" iyy="0.08" iyz="0" izz="0.08"/>
         </inertial>
     </link>
-    <joint name="baseHinge" type="continuous">
+    <joint name="interArm" type="revolute">
         <axis rpy="0 0 0" xyz="0 0 1"/>
-        <parent link="base"/>
-        <child link="arm1"/>
-    </joint>
-    <link name="arm2">
-        <visual>
-            <geometry>
-                <box size="1 .05 .05"/>
-            </geometry>
-            <origin rpy="0 0 0" xyz="0.5 0 0"/>
-            <material name="black"/>
-        </visual>
-        <collision>
-            <geometry>
-                <box size="1 .05 .05"/>
-            </geometry>
-            <origin rpy="0 0 0" xyz="0.5 0 0"/>
-        </collision>
-        <inertial>
-            <origin rpy="0 0 0" xyz="0.5 0 0"/>
-            <mass value="1.0"/>
-            <inertia ixx="0.001" ixy="0" ixz="0" iyy="0.08" iyz="0" izz="0.08"/>
-        </inertial>
-    </link>
-    <joint name="interArm" type="continuous">
-        <axis rpy="0 0 0" xyz="0 0 1"/>
+        <limit effort="30.0" velocity="1.0" lower="-3.14159" upper="3.14159"/>
         <parent link="arm1"/>
         <child link="arm2"/>
-        <origin rpy="0 0 0" xyz="1 0 0"/>
+        <origin rpy="0 0 0" xyz="0.75 0 0"/>
     </joint>
     <link name="endEffector">

File: src/daadbot_desc/urdf/2_link_urdf/2link_ros2_control.xacro (robot description, xacro)
@@ -23,6 +23,6 @@
         <joint name="baseHinge">
             <command_interface name="effort">
-                <param name="min">-15</param>
-                <param name="max">15</param>
+                <param name="min">-50</param>
+                <param name="max">50</param>
             </command_interface>
             <state_interface name="position"/>
@@ -32,6 +32,6 @@
         <joint name="interArm">
             <command_interface name="effort">
-                <param name="min">-15</param>
-                <param name="max">15</param>
+                <param name="min">-30</param>
+                <param name="max">30</param>
             </command_interface>
             <state_interface name="position"/>

Commit message: Tuned the gains for the 2 DOF CLF-CBF. Visualized the trajectory in gazebo and rviz

File: src/daadbot_desc/urdf/2_link_urdf/2link_robot.urdf.xacro (robot description, xacro)
@@ -46,5 +46,5 @@
     <joint name="baseHinge" type="revolute">
         <axis rpy="0 0 0" xyz="0 0 1"/>
-        <limit effort="50.0" velocity="1.0" lower="-3.14159" upper="3.14159"/>
+        <limit effort="50.0" velocity="1.0" lower="-1000.0" upper="1000.0"/>
         <parent link="base"/>
         <child link="arm1"/>
@@ -72,5 +72,5 @@
     <joint name="interArm" type="revolute">
         <axis rpy="0 0 0" xyz="0 0 1"/>
-        <limit effort="30.0" velocity="1.0" lower="-3.14159" upper="3.14159"/>
+        <limit effort="30.0" velocity="1.0" lower="-1000.0" upper="1000.0"/>
         <parent link="arm1"/>
         <child link="arm2"/>
