Commit message: Tuned the gains for the optimizer solver to work with the large quantile value. Added noise in masses+inertias+com in the noisy urdf. Can see the effect of 1. only FBL without CLF. 2. CLF with or without quantile (regular vs CR)

File: src/daadbot_desc/urdf/2_link_urdf/2link_robot_noisy_3.urdf (robot description, URDF)
Before this commit: robot 2link_robot, 5 links, 4 joints
Links:
- link arm1: mass 2.0 -> 3.000000
- link arm2: mass 1.5 -> 0.750000
